File: PCB/K-0.kicad_pcb (KiCad board)
At the start: 2 copper layers, 375.5 x 115.5 mm, 188 parts, among them IC1 BQ24040DSQR, IC2 TPS63031DSKR, J1 Display, J2 UJ20-C-H-G-MSMT-4B-P16-TR, J3 Battery, J4 PG_LED, J5 CHRG_LED, J6 POWER_LED, J7 Mode Selector, J8 Mode Selector, SW1 RotaryEncoder_Switch, SW10 A, SW11 Z, SW12 WIN, SW13 F1, SW14 2, SW15 W, SW16 S, SW17 X, SW18 LALT, SW19 F2, SW2 ESC, SW20 3, SW21 E, SW22 D, SW23 C, SW24 SPACE, SW25 F3, SW26 4, SW27 R, SW28 F, SW29 V, SW3 TILDE, SW30 F4, SW31 5, SW32 T, SW33 G, SW34 B, SW35 6, SW36 Y, SW37 H, SW38 N, SW39 F5, SW4 TAB, SW40 7, SW41 U, SW42 J, SW43 M, SW44 F6, SW45 8, SW46 I, SW47 K, SW48 COMMA, SW49 RALT, SW5 CAPS, SW50 F7, SW51 9, SW52 O, SW53 L, SW54 DOT, SW55 FN, SW56 F8, SW57 0, SW58 P, SW59 SEMICOLON, SW6 LSHIFT, SW60 SLASH, SW61 MENU, SW62 MINUS, SW63 SQBOPEN, SW64 QUOTE, SW65 RSHIFT, SW66 RCTRL, SW67 F9, SW68 EQUAL, SW69 SQBCLOSE, SW7 LCTRL, SW70 ENTER, SW71 UP, SW72 LEFT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

Commit message: layout rev1
Parts:
- removed D71, D72, D76, D78, D79, D80: 1N4148WS, Diode_SMD:D_SOD-323F
- removed J3: Battery, Connector_PinHeader_2.54mm:PinHeader_1x02_P2.54mm_Vertical
- removed SW71: UP, Button_Switch_Keyboard:SW_Cherry_MX_1.00u_PCB
- removed SW72: LEFT, Button_Switch_Keyboard:SW_Cherry_MX_1.00u_PCB
- removed SW76: DOWN, Button_Switch_Keyboard:SW_Cherry_MX_1.00u_PCB
- removed SW78: PRTSCR, Button_Switch_Keyboard:SW_Cherry_MX_1.00u_PCB
- removed SW79: DEL, Button_Switch_Keyboard:SW_Cherry_MX_1.00u_PCB
- removed SW80: RIGHT, Button_Switch_Keyboard:SW_Cherry_MX_1.00u_PCB
- J2: value UJ20-C-H-G-MSMT-4B-P16-TR -> USB4216-03-A; footprint usbc_lion:UJ20CHGMSMT4BP16TR -> usbc-lion:USB421603A
- J8: footprint Connector_PinHeader_2.54mm:PinHeader_1x03_P2.54mm_Vertical -> Connector_PinHeader_2.54mm:PinHeader_1x04_P2.54mm_Vertical
- moved SW1 376.8 mm to (401.0, 122.1)
- moved R3 375.5 mm to (328.9, 119.8)
- moved R4 374.9 mm to (332.6, 119.8)
- moved R5 374.2 mm to (336.3, 119.8)
- moved IC1 344.9 mm to (323.8, 122.5)
- moved C2 341.8 mm to (324.5, 120.6), turned to 180 degrees
- moved C1 337.3 mm to (321.1, 121.7), turned to 180 degrees
- moved C5 332.7 mm to (313.9, 129.7)
- moved C4 330.2 mm to (308.6, 126.8), turned to 90 degrees
- moved C3 329.3 mm to (309.6, 126.8), turned to 90 degrees
- moved IC2 328.2 mm to (310.9, 129.4)
- moved L2 327.8 mm to (305.4, 129.3), turned to 90 degrees
- moved J6 306.5 mm to (333.8, 129.8), turned to 90 degrees
- moved J5 301.0 mm to (326.2, 129.8), turned to 90 degrees
- moved R8 297.5 mm to (333.8, 126.0)
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Connections:
- D64 pad 1: Net-(D64-K) -> Net-(D12-K)
- D65 pad 1: Net-(D65-K) -> Net-(D12-K)
- D65 pad 2: Net-(D64-K) -> Net-(D12-K)
- D66 pad 2: Net-(D65-K) -> Net-(D12-K)
- D74 pad 1: Net-(D74-K) -> Net-(D12-K)
- D75 pad 2: Net-(D74-K) -> Net-(D12-K)
- D77 pad 1: Net-(D12-K) -> Net-(D77-K)
- D81 pad 2: /COL_16 -> Net-(D77-K)
- MDBT50Q_1 pad 9: /COL_16 -> unconnected-(MDBT50Q_1-P0.03/AIN1-Pad9)
- SW65 pad 2: Net-(D64-K) -> Net-(D12-K)
- SW66 pad 2: Net-(D65-K) -> Net-(D12-K)
- SW75 pad 2: Net-(D74-K) -> Net-(D12-K)
- SW81 pad 1: /COL_15 -> Net-(D73-K)
- SW81 pad 2: /COL_16 -> Net-(D77-K)
Other:
- board size 375.5 x 115.5 mm -> 286.2 x 129.2 mm
- board text added: "(NOT ON PCB, WILL BE RAISED UP)"
- board text added: "+"
- board text added: "-"
- board text added: "BAT"
- board text added: "DISPLAY_MODULE"

Commit message: schematics update + routing progress
Parts:
- moved C5 0.36 mm to (314.1, 129.9)
Connections:
- D10 pad 1: Net-(D10-K) -> /ROW_04
- D11 pad 1: Net-(D11-K) -> /ROW_05
- D11 pad 2: Net-(D10-K) -> Net-(D11-A)
- D12 pad 1: Net-(D12-K) -> /ROW_06
- D12 pad 2: Net-(D11-K) -> Net-(D12-A)
- D13 pad 1: Net-(D13-K) -> /ROW_01
- D13 pad 2: /COL_03 -> Net-(D13-A)
- D14 pad 1: Net-(D14-K) -> /ROW_02
- D14 pad 2: Net-(D13-K) -> Net-(D14-A)
- D15 pad 1: Net-(D15-K) -> /ROW_03
- D15 pad 2: Net-(D14-K) -> Net-(D15-A)
- D16 pad 1: Net-(D16-K) -> /ROW_04
- D16 pad 2: Net-(D15-K) -> Net-(D16-A)
- D17 pad 1: Net-(D17-K) -> /ROW_05
- D17 pad 2: Net-(D16-K) -> Net-(D17-A)
- D18 pad 1: Net-(D12-K) -> /ROW_06
- D18 pad 2: Net-(D17-K) -> Net-(D18-A)
- D19 pad 1: Net-(D19-K) -> /ROW_01
- D19 pad 2: /COL_04 -> Net-(D19-A)
- D2 pad 1: Net-(D2-K) -> /ROW_01
- D2 pad 2: /COL_01 -> Net-(D2-A)
- D20 pad 1: Net-(D20-K) -> /ROW_02
- D20 pad 2: Net-(D19-K) -> Net-(D20-A)
- D21 pad 1: Net-(D21-K) -> /ROW_03
- D21 pad 2: Net-(D20-K) -> Net-(D21-A)
- D22 pad 1: Net-(D22-K) -> /ROW_04
- D22 pad 2: Net-(D21-K) -> Net-(D22-A)
- D23 pad 1: Net-(D12-K) -> /ROW_05
- D23 pad 2: Net-(D22-K) -> Net-(D23-A)
- D24 pad 1: Net-(D12-K) -> /ROW_06
- D24 pad 2: Net-(D12-K) -> Net-(D24-A)
- D25 pad 1: Net-(D25-K) -> /ROW_01
- D25 pad 2: /COL_05 -> Net-(D25-A)
- D26 pad 1: Net-(D26-K) -> /ROW_02
- D26 pad 2: Net-(D25-K) -> Net-(D26-A)
- D27 pad 1: Net-(D27-K) -> /ROW_03
- D27 pad 2: Net-(D26-K) -> Net-(D27-A)
- D28 pad 1: Net-(D28-K) -> /ROW_04
- D28 pad 2: Net-(D27-K) -> Net-(D28-A)
- D29 pad 1: Net-(D12-K) -> /ROW_05
- D29 pad 2: Net-(D28-K) -> Net-(D29-A)
- D3 pad 1: Net-(D3-K) -> /ROW_02
- D3 pad 2: Net-(D2-K) -> Net-(D3-A)
- D30 pad 1: Net-(D30-K) -> /ROW_01
- D30 pad 2: /COL_06 -> Net-(D30-A)
- D31 pad 1: Net-(D31-K) -> /ROW_02
- D31 pad 2: Net-(D30-K) -> Net-(D31-A)
- D32 pad 1: Net-(D32-K) -> /ROW_03
- D32 pad 2: Net-(D31-K) -> Net-(D32-A)
- D33 pad 1: Net-(D33-K) -> /ROW_04
- D33 pad 2: Net-(D32-K) -> Net-(D33-A)
- D34 pad 1: Net-(D12-K) -> /ROW_05
- D34 pad 2: Net-(D33-K) -> Net-(D34-A)
- D35 pad 1: Net-(D35-K) -> /ROW_02
- D35 pad 2: /COL_06 -> Net-(D35-A)
- D36 pad 1: Net-(D36-K) -> /ROW_03
- D36 pad 2: Net-(D35-K) -> Net-(D36-A)
- D37 pad 1: Net-(D37-K) -> /ROW_04
- D37 pad 2: Net-(D36-K) -> Net-(D37-A)
- D38 pad 1: Net-(D12-K) -> /ROW_05
- D38 pad 2: Net-(D37-K) -> Net-(D38-A)
- D39 pad 1: Net-(D39-K) -> /ROW_01
- D39 pad 2: /COL_08 -> Net-(D39-A)
- D4 pad 1: Net-(D4-K) -> /ROW_03
- D4 pad 2: Net-(D3-K) -> Net-(D4-A)
- D40 pad 1: Net-(D40-K) -> /ROW_02
- D40 pad 2: Net-(D39-K) -> Net-(D40-A)
- D41 pad 1: Net-(D41-K) -> /ROW_03
- D41 pad 2: Net-(D40-K) -> Net-(D41-A)
- D42 pad 1: Net-(D42-K) -> /ROW_04
- D42 pad 2: Net-(D41-K) -> Net-(D42-A)
- D43 pad 1: Net-(D12-K) -> /ROW_05
- D43 pad 2: Net-(D42-K) -> Net-(D43-A)
- D44 pad 1: Net-(D44-K) -> /ROW_01
- D44 pad 2: /COL_09 -> Net-(D44-A)
- D45 pad 1: Net-(D45-K) -> /ROW_02
- D45 pad 2: Net-(D44-K) -> Net-(D45-A)
- D46 pad 1: Net-(D46-K) -> /ROW_03
- D46 pad 2: Net-(D45-K) -> Net-(D46-A)
- D47 pad 1: Net-(D47-K) -> /ROW_04
- D47 pad 2: Net-(D46-K) -> Net-(D47-A)
- D48 pad 1: Net-(D48-K) -> /ROW_05
- D48 pad 2: Net-(D47-K) -> Net-(D48-A)
- D49 pad 1: Net-(D12-K) -> /ROW_06
- D49 pad 2: Net-(D48-K) -> Net-(D49-A)
- D5 pad 1: Net-(D5-K) -> /ROW_04
- D5 pad 2: Net-(D4-K) -> Net-(D5-A)
- D50 pad 1: Net-(D50-K) -> /ROW_01
- D50 pad 2: /COL_10 -> Net-(D50-A)
- D51 pad 1: Net-(D51-K) -> /ROW_02
- D51 pad 2: Net-(D50-K) -> Net-(D51-A)
- D52 pad 1: Net-(D52-K) -> /ROW_03
- D52 pad 2: Net-(D51-K) -> Net-(D52-A)
- D53 pad 1: Net-(D53-K) -> /ROW_04
- D53 pad 2: Net-(D52-K) -> Net-(D53-A)
- D54 pad 1: Net-(D54-K) -> /ROW_05
- D54 pad 2: Net-(D53-K) -> Net-(D54-A)
- D55 pad 1: Net-(D12-K) -> /ROW_06
- D55 pad 2: Net-(D54-K) -> Net-(D55-A)
- D56 pad 1: Net-(D56-K) -> /ROW_01
- D56 pad 2: /COL_11 -> Net-(D56-A)
- D57 pad 1: Net-(D57-K) -> /ROW_02
- D57 pad 2: Net-(D56-K) -> Net-(D57-A)
- D58 pad 1: Net-(D58-K) -> /ROW_03
- D58 pad 2: Net-(D57-K) -> Net-(D58-A)
- D59 pad 1: Net-(D59-K) -> /ROW_04
- D59 pad 2: Net-(D58-K) -> Net-(D59-A)
- D6 pad 1: Net-(D6-K) -> /ROW_05
- D6 pad 2: Net-(D5-K) -> Net-(D6-A)
- D60 pad 1: Net-(D60-K) -> /ROW_05
- D60 pad 2: Net-(D59-K) -> Net-(D60-A)
- D61 pad 1: Net-(D12-K) -> /ROW_06
- D61 pad 2: Net-(D60-K) -> Net-(D61-A)
- D62 pad 1: Net-(D62-K) -> /ROW_02
- D62 pad 2: /COL_11 -> Net-(D62-A)
- D63 pad 1: Net-(D63-K) -> /ROW_03
- D63 pad 2: Net-(D62-K) -> Net-(D63-A)
- D64 pad 1: Net-(D12-K) -> /ROW_04
- D64 pad 2: Net-(D63-K) -> Net-(D64-A)
- D65 pad 1: Net-(D12-K) -> /ROW_05
- D65 pad 2: Net-(D12-K) -> Net-(D65-A)
- D66 pad 1: Net-(D12-K) -> /ROW_06
- D66 pad 2: Net-(D12-K) -> Net-(D66-A)
- D67 pad 1: Net-(D67-K) -> /ROW_01
- D67 pad 2: /COL_13 -> Net-(D67-A)
- D68 pad 1: Net-(D68-K) -> /ROW_02
- D68 pad 2: Net-(D67-K) -> Net-(D68-A)
- D69 pad 1: Net-(D12-K) -> /ROW_03
- D69 pad 2: Net-(D68-K) -> Net-(D69-A)
- D7 pad 1: Net-(D12-K) -> /ROW_06
- D7 pad 2: Net-(D6-K) -> Net-(D7-A)
- D70 pad 1: Net-(D12-K) -> /ROW_04
- D70 pad 2: Net-(D12-K) -> Net-(D70-A)
- D73 pad 1: Net-(D73-K) -> /ROW_01
- D73 pad 2: /COL_14 -> Net-(D73-A)
- D74 pad 1: Net-(D12-K) -> /ROW_02
- D74 pad 2: Net-(D73-K) -> Net-(D74-A)
- D75 pad 1: Net-(D12-K) -> /ROW_03
- D75 pad 2: Net-(D12-K) -> Net-(D75-A)
- D77 pad 1: Net-(D77-K) -> /ROW_01
- D77 pad 2: /COL_15 -> Net-(D77-A)
- D8 pad 1: Net-(D8-K) -> /ROW_02
- D8 pad 2: /COL_01 -> Net-(D8-A)
- D81 pad 1: Net-(D12-K) -> /ROW_02
- D81 pad 2: Net-(D77-K) -> Net-(D81-A)
- D9 pad 1: Net-(D10-A) -> /ROW_03
- D9 pad 2: Net-(D8-K) -> Net-(D9-A)
- MDBT50Q_1 pad 5: /COL_11 -> /COL_12
- MDBT50Q_1 pad 50: /COL_01 -> /COL_02
- MDBT50Q_1 pad 58: /COL_06 -> /COL_07
- SW10 pad 1: Net-(D4-K) -> /COL_02
- SW11 pad 1: Net-(D5-K) -> /COL_02
- SW11 pad 2: Net-(D10-K) -> Net-(D11-A)
- SW12 pad 1: Net-(D6-K) -> /COL_02
- SW12 pad 2: Net-(D11-K) -> Net-(D12-A)
- SW13 pad 1: /COL_01 -> /COL_03
- SW13 pad 2: /COL_03 -> Net-(D13-A)
- SW14 pad 1: /COL_01 -> /COL_03
- SW14 pad 2: Net-(D13-K) -> Net-(D14-A)
- SW15 pad 1: Net-(D8-K) -> /COL_03
- SW15 pad 2: Net-(D14-K) -> Net-(D15-A)
- SW16 pad 1: Net-(D10-A) -> /COL_03
- SW16 pad 2: Net-(D15-K) -> Net-(D16-A)
- SW17 pad 1: Net-(D10-K) -> /COL_03
- SW17 pad 2: Net-(D16-K) -> Net-(D17-A)
- SW18 pad 1: Net-(D11-K) -> /COL_03
- SW18 pad 2: Net-(D17-K) -> Net-(D18-A)
- SW19 pad 1: /COL_03 -> /COL_04
- SW19 pad 2: /COL_04 -> Net-(D19-A)
- SW2 pad 1: /ROW_01 -> /COL_01
- SW2 pad 2: /COL_01 -> Net-(D2-A)
- SW20 pad 1: Net-(D13-K) -> /COL_04
- SW20 pad 2: Net-(D19-K) -> Net-(D20-A)
- SW21 pad 1: Net-(D14-K) -> /COL_04
- SW21 pad 2: Net-(D20-K) -> Net-(D21-A)
- SW22 pad 1: Net-(D15-K) -> /COL_04
- SW22 pad 2: Net-(D21-K) -> Net-(D22-A)
- SW23 pad 1: Net-(D16-K) -> /COL_04
- SW23 pad 2: Net-(D22-K) -> Net-(D23-A)
- SW24 pad 1: Net-(D17-K) -> /COL_04
- SW24 pad 2: Net-(D12-K) -> Net-(D24-A)
- SW25 pad 1: /COL_04 -> /COL_05
- SW25 pad 2: /COL_05 -> Net-(D25-A)
- SW26 pad 1: Net-(D19-K) -> /COL_05
- SW26 pad 2: Net-(D25-K) -> Net-(D26-A)
- SW27 pad 1: Net-(D20-K) -> /COL_05
- SW27 pad 2: Net-(D26-K) -> Net-(D27-A)
- SW28 pad 1: Net-(D21-K) -> /COL_05
- SW28 pad 2: Net-(D27-K) -> Net-(D28-A)
- SW29 pad 1: Net-(D22-K) -> /COL_05
- SW29 pad 2: Net-(D28-K) -> Net-(D29-A)
- SW3 pad 1: /ROW_02 -> /COL_01
- SW3 pad 2: Net-(D2-K) -> Net-(D3-A)
- SW30 pad 1: /COL_05 -> /COL_06
- SW30 pad 2: /COL_06 -> Net-(D30-A)
- SW31 pad 1: Net-(D25-K) -> /COL_06
- SW31 pad 2: Net-(D30-K) -> Net-(D31-A)
- SW32 pad 1: Net-(D26-K) -> /COL_06
- SW32 pad 2: Net-(D31-K) -> Net-(D32-A)
- SW33 pad 1: Net-(D27-K) -> /COL_06
- SW33 pad 2: Net-(D32-K) -> Net-(D33-A)
- SW34 pad 1: Net-(D28-K) -> /COL_06
- SW34 pad 2: Net-(D33-K) -> Net-(D34-A)
- SW35 pad 1: Net-(D30-K) -> /COL_07
- SW35 pad 2: /COL_06 -> Net-(D35-A)
- SW36 pad 1: Net-(D31-K) -> /COL_07
- SW36 pad 2: Net-(D35-K) -> Net-(D36-A)
- SW37 pad 1: Net-(D32-K) -> /COL_07
- SW37 pad 2: Net-(D36-K) -> Net-(D37-A)
- SW38 pad 1: Net-(D33-K) -> /COL_07
- SW38 pad 2: Net-(D37-K) -> Net-(D38-A)
- SW39 pad 1: /COL_06 -> /COL_08
- SW39 pad 2: /COL_08 -> Net-(D39-A)
- SW4 pad 1: /ROW_03 -> /COL_01
- SW4 pad 2: Net-(D3-K) -> Net-(D4-A)
- SW40 pad 1: /COL_06 -> /COL_08
- SW40 pad 2: Net-(D39-K) -> Net-(D40-A)
- SW41 pad 1: Net-(D35-K) -> /COL_08
- SW41 pad 2: Net-(D40-K) -> Net-(D41-A)
- SW42 pad 1: Net-(D36-K) -> /COL_08
- SW42 pad 2: Net-(D41-K) -> Net-(D42-A)
- SW43 pad 1: Net-(D37-K) -> /COL_08
- SW43 pad 2: Net-(D42-K) -> Net-(D43-A)
- SW44 pad 1: /COL_08 -> /COL_09
- SW44 pad 2: /COL_09 -> Net-(D44-A)
- SW45 pad 1: Net-(D39-K) -> /COL_09
- SW45 pad 2: Net-(D44-K) -> Net-(D45-A)
- SW46 pad 1: Net-(D40-K) -> /COL_09
- SW46 pad 2: Net-(D45-K) -> Net-(D46-A)
- SW47 pad 1: Net-(D41-K) -> /COL_09
- SW47 pad 2: Net-(D46-K) -> Net-(D47-A)
- SW48 pad 1: Net-(D42-K) -> /COL_09
- SW48 pad 2: Net-(D47-K) -> Net-(D48-A)
- SW49 pad 1: Net-(D12-K) -> /COL_09
- SW49 pad 2: Net-(D48-K) -> Net-(D49-A)
- SW5 pad 1: /ROW_04 -> /COL_01
- SW5 pad 2: Net-(D4-K) -> Net-(D5-A)
- SW50 pad 1: /COL_09 -> /COL_10
- SW50 pad 2: /COL_10 -> Net-(D50-A)
- SW51 pad 1: Net-(D44-K) -> /COL_10
- SW51 pad 2: Net-(D50-K) -> Net-(D51-A)
- SW52 pad 1: Net-(D45-K) -> /COL_10
- SW52 pad 2: Net-(D51-K) -> Net-(D52-A)
- SW53 pad 1: Net-(D46-K) -> /COL_10
- SW53 pad 2: Net-(D52-K) -> Net-(D53-A)
- SW54 pad 1: Net-(D47-K) -> /COL_10
- SW54 pad 2: Net-(D53-K) -> Net-(D54-A)
- SW55 pad 1: Net-(D48-K) -> /COL_10
- SW55 pad 2: Net-(D54-K) -> Net-(D55-A)
- SW56 pad 1: /COL_10 -> /COL_11
- SW56 pad 2: /COL_11 -> Net-(D56-A)
- SW57 pad 1: Net-(D50-K) -> /COL_11
- SW57 pad 2: Net-(D56-K) -> Net-(D57-A)
- SW58 pad 1: Net-(D51-K) -> /COL_11
- SW58 pad 2: Net-(D57-K) -> Net-(D58-A)
- SW59 pad 1: Net-(D52-K) -> /COL_11
- SW59 pad 2: Net-(D58-K) -> Net-(D59-A)
- SW6 pad 1: /ROW_05 -> /COL_01
- SW6 pad 2: Net-(D5-K) -> Net-(D6-A)
- SW60 pad 1: Net-(D53-K) -> /COL_11
- SW60 pad 2: Net-(D59-K) -> Net-(D60-A)
- SW61 pad 1: Net-(D54-K) -> /COL_11
- SW61 pad 2: Net-(D60-K) -> Net-(D61-A)
- SW62 pad 1: Net-(D56-K) -> /COL_12
- SW62 pad 2: /COL_11 -> Net-(D62-A)
- SW63 pad 1: Net-(D57-K) -> /COL_12
- SW63 pad 2: Net-(D62-K) -> Net-(D63-A)
- SW64 pad 1: Net-(D58-K) -> /COL_12
- SW64 pad 2: Net-(D63-K) -> Net-(D64-A)
- SW65 pad 1: Net-(D59-K) -> /COL_12
- SW65 pad 2: Net-(D12-K) -> Net-(D65-A)
- SW66 pad 1: Net-(D60-K) -> /COL_12
- SW66 pad 2: Net-(D12-K) -> Net-(D66-A)
- SW67 pad 1: /COL_11 -> /COL_13
- SW67 pad 2: /COL_13 -> Net-(D67-A)
- SW68 pad 1: /COL_11 -> /COL_13
- SW68 pad 2: Net-(D67-K) -> Net-(D68-A)
- SW69 pad 1: Net-(D62-K) -> /COL_13
- SW69 pad 2: Net-(D68-K) -> Net-(D69-A)
- SW7 pad 1: /ROW_06 -> /COL_01
- SW7 pad 2: Net-(D6-K) -> Net-(D7-A)
- SW70 pad 1: Net-(D63-K) -> /COL_13
- SW70 pad 2: Net-(D12-K) -> Net-(D70-A)
- SW73 pad 1: /COL_13 -> /COL_14
- SW73 pad 2: /COL_14 -> Net-(D73-A)
- SW74 pad 1: Net-(D67-K) -> /COL_14
- SW74 pad 2: Net-(D73-K) -> Net-(D74-A)
- SW75 pad 1: Net-(D68-K) -> /COL_14
- SW75 pad 2: Net-(D12-K) -> Net-(D75-A)
- SW77 pad 1: /COL_14 -> /COL_15
- SW77 pad 2: /COL_15 -> Net-(D77-A)
- SW8 pad 1: Net-(D2-K) -> /COL_02
- SW8 pad 2: /COL_01 -> Net-(D8-A)
- SW81 pad 1: Net-(D73-K) -> /COL_15
- SW81 pad 2: Net-(D77-K) -> Net-(D81-A)
- SW9 pad 1: Net-(D3-K) -> /COL_02
- SW9 pad 2: Net-(D8-K) -> Net-(D9-A)
Routing:
- net /ROW_04: track 0.00 -> 417.8 mm, vias 0 -> 4
- net /ROW_03: track 0.00 -> 397.6 mm, vias 0 -> 2
- net /ROW_02: track 0.00 -> 365.5 mm, vias 0 -> 2
- net /ROW_05: track 0.00 -> 360.9 mm, vias 0 -> 2
- net /ROW_01: track 0.00 -> 285.6 mm, vias 0 -> 2
- net /ROW_06: track 0.00 -> 278.8 mm, vias 0 -> 2
- net /USB_D+: track 0.00 -> 206.3 mm, vias 0 -> 2
- net /USB_D-: track 0.00 -> 206.1 mm, vias 0 -> 2
- net /MODE_SEL_PIN: track 0.00 -> 158.2 mm
- net /VIN_MEASURE: track 0.00 -> 136.9 mm
- net /COL_04: track 0.00 -> 134.4 mm
- net /COL_11: track 0.00 -> 124.1 mm
- net /COL_10: track 0.00 -> 119.3 mm
- net /COL_09: track 0.00 -> 116.0 mm
- net /COL_03: track 0.00 -> 110.0 mm
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Other:
- board size 286.2 x 129.2 mm -> 286.2 x 129.4 mm
- copper layers 2 -> 4

Commit message: routing almost finished
Parts:
- added J3: ProgConn, Connector_PinHeader_2.54mm:PinHeader_1x04_P2.54mm_Vertical, F.Cu at (370.7, 119.0)
- moved J7 160.8 mm to (354.2, 119.0)
- moved C1 0.73 mm to (321.5, 121.1), turned to 90 degrees
Connections:
- MDBT50Q_1 pad 13: /ROW_06 -> /COL_01
- MDBT50Q_1 pad 14: unconnected-(MDBT50Q_1-P0.30/AIN6-Pad14) -> /COL_02
- MDBT50Q_1 pad 16: /ROW_05 -> /COL_03
- MDBT50Q_1 pad 17: unconnected-(MDBT50Q_1-P0.00/XL1-Pad17) -> /COL_04
- MDBT50Q_1 pad 18: unconnected-(MDBT50Q_1-P0.01/XL2-Pad18) -> /COL_05
- MDBT50Q_1 pad 19: /ROW_04 -> /COL_06
- MDBT50Q_1 pad 20: unconnected-(MDBT50Q_1-P0.04/AIN2-Pad20) -> /COL_07
- MDBT50Q_1 pad 21: unconnected-(MDBT50Q_1-P0.05/AIN3-Pad21) -> /COL_08
- MDBT50Q_1 pad 22: unconnected-(MDBT50Q_1-P0.06-Pad22) -> /COL_09
- MDBT50Q_1 pad 23: unconnected-(MDBT50Q_1-P0.07-Pad23) -> /COL_10
- MDBT50Q_1 pad 24: unconnected-(MDBT50Q_1-P0.08-Pad24) -> /COL_11
- MDBT50Q_1 pad 25: /COL_08 -> /COL_12
- MDBT50Q_1 pad 26: /COL_09 -> /COL_13
- MDBT50Q_1 pad 27: unconnected-(MDBT50Q_1-P0.11-Pad27) -> /COL_14
- MDBT50Q_1 pad 29: unconnected-(MDBT50Q_1-P0.12-Pad29) -> /COL_15
- MDBT50Q_1 pad 3: /COL_10 -> unconnected-(MDBT50Q_1-P1.10-Pad3)
- MDBT50Q_1 pad 4: /COL_11 -> /ROW_01
- MDBT50Q_1 pad 45: /ROW_01 -> unconnected-(MDBT50Q_1-P0.23-Pad45)
- MDBT50Q_1 pad 48: /ROW_02 -> unconnected-(MDBT50Q_1-P0.24-Pad48)
- MDBT50Q_1 pad 49: /ROW_03 -> unconnected-(MDBT50Q_1-P0.25-Pad49)
- MDBT50Q_1 pad 5: /COL_12 -> /ROW_02
- MDBT50Q_1 pad 50: /COL_02 -> unconnected-(MDBT50Q_1-P1.02-Pad50)
- MDBT50Q_1 pad 56: /COL_04 -> unconnected-(MDBT50Q_1-P1.04-Pad56)
- MDBT50Q_1 pad 57: /COL_06 -> unconnected-(MDBT50Q_1-P1.06-Pad57)
- MDBT50Q_1 pad 58: /COL_07 -> unconnected-(MDBT50Q_1-P1.07-Pad58)
- MDBT50Q_1 pad 59: /COL_05 -> unconnected-(MDBT50Q_1-P1.05-Pad59)
- MDBT50Q_1 pad 6: /COL_13 -> /ROW_03
- MDBT50Q_1 pad 60: /COL_03 -> unconnected-(MDBT50Q_1-P1.03-Pad60)
- MDBT50Q_1 pad 61: /COL_01 -> unconnected-(MDBT50Q_1-P1.01-Pad61)
- MDBT50Q_1 pad 7: /COL_14 -> /ROW_04
- MDBT50Q_1 pad 8: /COL_15 -> /ROW_05
- MDBT50Q_1 pad 9: unconnected-(MDBT50Q_1-P0.03/AIN1-Pad9) -> /ROW_06
Routing:
- net /COL_01: track 104.1 -> 308.9 mm, vias 0 -> 1
- net /COL_02: track 95.1 -> 293.3 mm, vias 0 -> 3
- net VBUS: track 29.5 -> 224.2 mm, vias 0 -> 2
- net /COL_03: track 110.0 -> 273.4 mm
- net /+BAT: track 1.17 -> 155.9 mm, vias 0 -> 1
- net /POWER: track 0.00 -> 149.9 mm, vias 0 -> 1
- net /MODE_SEL_PIN: track 158.2 -> 10.9 mm, vias 0 -> 1
- net /COL_04: track 134.4 -> 278.9 mm
- net /ROW_06: track 278.8 -> 419.4 mm, vias 2 -> 3
- net /COL_06: track 67.0 -> 196.4 mm, vias 0 -> 2
- net /COL_05: track 86.1 -> 212.2 mm
- net /COL_07: track 67.0 -> 175.4 mm, vias 0 -> 1
- net /COL_08: track 90.0 -> 172.3 mm, vias 0 -> 2
- net /ROW_04: track 417.8 -> 349.2 mm
- net /ROW_03: track 397.6 -> 334.5 mm, vias 2 -> 3
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- added copper zone on In2.Cu, net +3.3V
- added copper zone on B.Cu, net GND
- added copper zone on F.Cu, net GND
- added copper zone on In1.Cu, net GND
Other:
- board text added: "3V3/GND/SWDCLK/SWDIO"
- board text added: "3v3"
- board text added: "Programmer"

Commit message: pcb finished
Parts:
- added G***: LOGO, LOGO, F.Cu at (154.9, 147.3)
- added J9: LED_STRIP, Connector_PinHeader_2.54mm:PinHeader_1x03_P2.54mm_Vertical, F.Cu at (284.8, 236.4)
- SW10, SW11, SW13, SW14, SW15, SW16, SW17, SW19, SW2, SW20, SW21, SW22, SW23, SW25, SW26, SW27, SW28, SW29, SW3, SW30, SW31, SW32, SW33, SW34, SW35, SW36, SW37, SW38, SW39, SW40, SW41, SW42, SW43, SW44, SW45, SW46, SW47, SW48, SW50, SW51, SW52, SW53, SW54, SW56, SW57, SW58, SW59, SW60, SW62, SW63, SW64, SW67, SW68, SW69, SW73, SW77, SW8, SW81, SW9: footprint Button_Switch_Keyboard:SW_Cherry_MX_1.00u_PCB -> Button_Switch_Keyboard:3Dfyd_SW_Cherry_MX_1.00u_PCB
- SW12, SW18, SW49, SW55, SW61, SW66, SW7: footprint Button_Switch_Keyboard:SW_Cherry_MX_1.25u_PCB -> Button_Switch_Keyboard:3dfyd_SW_Cherry_MX_1.25u_PCB
- SW24: footprint Button_Switch_Keyboard:SW_Cherry_MX_6.25u_PCB -> Button_Switch_Keyboard:3Dfyd_SW_Cherry_MX_6.25u_PCB
- SW4, SW75: footprint Button_Switch_Keyboard:SW_Cherry_MX_1.50u_PCB -> Button_Switch_Keyboard:3Dfyd_SW_Cherry_MX_1.50u_PCB
- SW5: footprint Button_Switch_Keyboard:SW_Cherry_MX_1.75u_PCB -> Button_Switch_Keyboard:3Dfyd_SW_Cherry_MX_1.75u_PCB
- SW6, SW70: footprint Button_Switch_Keyboard:SW_Cherry_MX_2.25u_PCB -> Button_Switch_Keyboard:3Dfyd_SW_Cherry_MX_2.25u_PCB
- SW65: footprint Button_Switch_Keyboard:SW_Cherry_MX_2.75u_PCB -> Button_Switch_Keyboard:3Dfyd_SW_Cherry_MX_2.75u_PCB
- SW74: footprint Button_Switch_Keyboard:SW_Cherry_MX_2.00u_PCB -> Button_Switch_Keyboard:3Dfyd_SW_Cherry_MX_2.00u_PCB
Connections:
- MDBT50Q_1 pad 45: unconnected-(MDBT50Q_1-P0.23-Pad45) -> /LED_STRIP_CTRL
Routing:
- net /LED_STRIP_CTRL: track 0.00 -> 293.4 mm, vias 0 -> 1
- net VBUS: track 224.2 -> 354.6 mm
- net GND: track 47.3 -> 51.4 mm, vias 78 -> 408
- net /+BAT: track 155.9 -> 152.4 mm
- net /COL_12: track 133.8 -> 135.4 mm
- net /COL_14: track 91.7 -> 90.9 mm
Other:
- board size 286.2 x 129.4 mm -> 291.2 x 132.7 mm
- board text added: "3V3"
- board text added: "BLK"
- board text added: "D"
- board text added: "DISPLAY_CONN"
- board text added: "K-0"
- board text added: "MODE_SEL_SW"
- board text added: "POWER_SEL_SWITCH"
