File: PCB/K-0.kicad_sch (KiCad schematic)
At the start: 162 parts, among them J1 Display, SW1 RotaryEncoder_Switch, SW10 SW_Push, SW11 SW_Push, SW12 SW_Push, SW13 SW_Push, SW14 SW_Push, SW15 SW_Push, SW16 SW_Push, SW17 SW_Push, SW18 SW_Push, SW19 SW_Push, SW2 SW_Push, SW20 SW_Push, SW21 SW_Push, SW22 SW_Push, SW23 SW_Push, SW24 SW_Push, SW25 SW_Push, SW26 SW_Push, SW27 SW_Push, SW28 SW_Push, SW29 SW_Push, SW3 SW_Push, SW30 SW_Push, SW31 SW_Push, SW32 SW_Push, SW33 SW_Push, SW34 SW_Push, SW35 SW_Push, SW36 SW_Push, SW37 SW_Push, SW38 SW_Push, SW39 SW_Push, SW4 SW_Push, SW40 SW_Push, SW41 SW_Push, SW42 SW_Push, SW43 SW_Push, SW44 SW_Push, SW45 SW_Push, SW46 SW_Push, SW47 SW_Push, SW48 SW_Push, SW49 SW_Push, SW5 SW_Push, SW50 SW_Push, SW51 SW_Push, SW52 SW_Push, SW53 SW_Push, SW54 SW_Push, SW55 SW_Push, SW56 SW_Push, SW57 SW_Push, SW58 SW_Push, SW59 SW_Push, SW6 SW_Push, SW60 SW_Push, SW61 SW_Push, SW62 SW_Push, SW63 SW_Push, SW64 SW_Push, SW65 SW_Push, SW66 SW_Push, SW67 SW_Push, SW68 SW_Push, SW69 SW_Push, SW7 SW_Push, SW70 SW_Push, SW71 SW_Push, SW72 SW_Push, SW73 SW_Push, SW74 SW_Push, SW75 SW_Push, SW76 SW_Push, SW77 SW_Push, SW78 SW_Push, SW79 SW_Push, SW8 SW_Push, SW80 SW_Push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

Commit message: added footprints for display connector and know
Parts:
- J1: footprint (none) -> Connector_PinHeader_2.54mm:PinHeader_1x08_P2.54mm_Vertical
- SW1: footprint (none) -> Rotary_Encoder:RotaryEncoder_Alps_EC11E-Switch_Vertical_H20mm
Changed lines of the file:
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@@
 			)
 		)
-		(property "Footprint" ""
+		(property "Footprint" "Connector_PinHeader_2.54mm:PinHeader_1x08_P2.54mm_Vertical"
 			(at 34.29 50.8 0)
 			(effects
@@
 			)
 		)
-		(property "Footprint" ""
+		(property "Footprint" "Rotary_Encoder:RotaryEncoder_Alps_EC11E-Switch_Vertical_H20mm"
 			(at 92.71 44.196 0)
 			(effects

Commit message: finished schematics
Parts:
- added C1, C2: 1uF, Capacitor_SMD:C_0402_1005Metric, symbol Device:C_Small
- added C3, C4: 10uF, Capacitor_SMD:C_0402_1005Metric, symbol Device:C_Small
- added C5: 0.1uF, Capacitor_SMD:C_0402_1005Metric, symbol Device:C_Small
- added IC1: BQ24040DSQR, BQ24040DSQR-lion:SON40P200X200X80-11N, symbol BQ24040DSQR:BQ24040DSQR
- added IC2: TPS63031DSKR, TPS63031DSKR-lion:SON50P250X250X80-11N-D, symbol TPS63031DSKR:TPS63031DSKR
- added J2: UJ20-C-H-G-MSMT-4B-P16-TR, usbc_lion:UJ20CHGMSMT4BP16TR, symbol UJ20-C-H-G-MSMT-4B-P16-TR:UJ20-C-H-G-MSMT-4B-P16-TR
- added J3: Battery, Connector_PinHeader_2.54mm:PinHeader_1x02_P2.54mm_Vertical, symbol Connector_Generic:Conn_01x02
- added J4: PG_LED, Connector_PinHeader_2.54mm:PinHeader_1x02_P2.54mm_Vertical, symbol Connector_Generic:Conn_01x02
- added J5: CHRG_LED, Connector_PinHeader_2.54mm:PinHeader_1x02_P2.54mm_Vertical, symbol Connector_Generic:Conn_01x02
- added J6: POWER_LED, Connector_PinHeader_2.54mm:PinHeader_1x02_P2.54mm_Vertical, symbol Connector_Generic:Conn_01x02
- added J7, J8: Mode Selector, Connector_PinHeader_2.54mm:PinHeader_1x03_P2.54mm_Vertical, symbol Connector_Generic:Conn_01x03
- added L2: LPS3015-222MRC, LPS3015-222MRC:IND_LPS3015-222MRC, symbol LPS3015-222MRC:LPS3015-222MRC
- added MDBT50Q_1: MDBT50Q_1, RF_Module:Raytac_MDBT50Q, symbol MDBT50Q-U_52840_230606:MDBT50Q_52840
- added R1, R2: 5.1k, Resistor_SMD:R_0402_1005Metric, symbol Device:R_Small
- added R10: 400k, Connector_PinHeader_2.54mm:PinHeader_1x02_P2.54mm_Vertical, symbol Device:R_Small
- added R3: 1k, Connector_PinHeader_2.54mm:PinHeader_1x02_P2.54mm_Vertical, symbol Device:R_Small
- added R4: 2k, Connector_PinHeader_2.54mm:PinHeader_1x02_P2.54mm_Vertical, symbol Device:R_Small
- added R5: 10k, Connector_PinHeader_2.54mm:PinHeader_1x02_P2.54mm_Vertical, symbol Device:R_Small
- added R6, R7, R8: 330, Connector_PinHeader_2.54mm:PinHeader_1x02_P2.54mm_Vertical, symbol Device:R_Small
- added R9: 300k, Connector_PinHeader_2.54mm:PinHeader_1x02_P2.54mm_Vertical, symbol Device:R_Small
- D1, D10, D11, D12, D13, D14, D15, D16, D17, D18, D19, D2, D20, D21, D22, D23, D24, D25, D26, D27, D28, D29, D3, D30, D31, D32, D33, D34, D35, D36, D37, D38, D39, D4, D40, D41, D42, D43, D44, D45, D46, D47, D48, D49, D5, D50, D51, D52, D53, D54, D55, D56, D57, D58, D59, D6, D60, D61, D62, D63, D64, D65, D66, D67, D68, D69, D7, D70, D71, D72, D73, D74, D75, D76, D77, D78, D79, D8, D80, D9: value D_Small -> 1N4148WS; footprint (none) -> Diode_SMD:D_SOD-323F; Manufacturer_Part_Number (none) -> 1N4148WS
Connections:
- net +3.3V: now also C3.1, C4.1, IC2.1 (VOUT), IC2.10 (FB), J7.3 (Pin_3), MDBT50Q_1.28 (VDD), MDBT50Q_1.30 (VDDH), R6.2, R7.2, R8.2
- net COL_01: now also MDBT50Q_1.61 (P1.01)
- net COL_02: now also MDBT50Q_1.50 (P1.02)
- net COL_03: now also MDBT50Q_1.60 (P1.03)
- net COL_04: now also MDBT50Q_1.56 (P1.04)
- net COL_05: now also MDBT50Q_1.59 (P1.05)
- net COL_06: now also MDBT50Q_1.57 (P1.06)
- net COL_07: now also MDBT50Q_1.58 (P1.07)
- net COL_08: now also MDBT50Q_1.25 (P1.08)
- net COL_09: now also MDBT50Q_1.26 (P1.09)
- net COL_10: now also MDBT50Q_1.3 (P1.10)
- net Display_BLK: now also MDBT50Q_1.42 (P0.19)
- net Display_CS: now also MDBT50Q_1.36 (P0.14)
- net Display_DC: now also MDBT50Q_1.41 (P0.17)
- net Display_MOSI: now also MDBT50Q_1.39 (P0.15)
- net Display_RES: now also MDBT50Q_1.38 (P0.16)
- net Display_SCLK: now also MDBT50Q_1.37 (P0.13)
- net GND: now also C1.2, C2.2, C3.2, C4.2, C5.2, IC1.11 (EP), IC1.3 (VSS), IC1.7 (ISET2), IC2.11 (EP), IC2.3 (PGND), IC2.9 (GND), J2.A1 (GND_1), J2.B1 (GND_2), J3.1 (Pin_1), J6.2 (Pin_2), J7.1 (Pin_1), MDBT50Q_1.1 (GND@1), MDBT50Q_1.15 (GND@15), MDBT50Q_1.2 (GND@2), MDBT50Q_1.33 (GND@33), MDBT50Q_1.55 (GND@55), R1.2, R10.1, R2.2, R3.2, R4.2, R5.2
- net RE_A: now also MDBT50Q_1.44 (P0.20)
- net RE_B: now also MDBT50Q_1.43 (P0.21)
- net RE_Sw: now also MDBT50Q_1.46 (P0.22)
- net ROW_01: now also MDBT50Q_1.45 (P0.23)
- net ROW_02: now also MDBT50Q_1.48 (P0.24)
- net ROW_03: now also MDBT50Q_1.49 (P0.25)
- net ROW_04: now also MDBT50Q_1.19 (P0.26)
- net ROW_05: now also MDBT50Q_1.16 (P0.27)
- net ROW_06: now also MDBT50Q_1.13 (P0.28/AIN4)
- net ROW_07: now also MDBT50Q_1.10 (P0.29/AIN5)
- net ROW_08: now also MDBT50Q_1.14 (P0.30/AIN6)
- new net: J5.1 (Pin_1), R7.1
- new net: J4.1 (Pin_1), R6.1
- new net: IC1.4 (PRETERM), R4.1
- new net: J6.1 (Pin_1), R8.1
- new net: IC1.2 (ISET), R3.1
- new net: IC1.9 (TS), R5.1
- new net: C5.1, IC2.6 (EN), IC2.7 (PS/SYNC), IC2.8 (VINA)
- new net +BAT: C2.1, IC1.10 (OUT), J3.2 (Pin_2), J8.3 (Pin_3)
- new net CHRG_LED: IC1.8 (~{CHG}), J5.2 (Pin_2)
- new net CHRG_PGLED: IC1.5 (~{PG}), J4.2 (Pin_2)
- new net MCU_RESET: MDBT50Q_1.40 (P0.18/RESET)
- new net MCU_SWDCLK: MDBT50Q_1.53 (SWDCLK)
- new net MCU_SWDIO: MDBT50Q_1.51 (SWDIO)
- new net MODE_SEL_PIN: J7.2 (Pin_2), MDBT50Q_1.47 (P1.00)
- new net POWER: IC2.5 (VIN), J8.2 (Pin_2), R9.2
- new net REG_L1: IC2.4 (L1), L2.1
- new net REG_L2: IC2.2 (L2), L2.2
- new net USB_CC1: J2.A5 (CC1), R1.1
- new net USB_CC2: J2.B5 (CC2), R2.1
- new net USB_D+: J2.A6 (DP1), J2.B6 (DP2), MDBT50Q_1.35 (D+)
- new net USB_D-: J2.A7 (DN1), J2.B7 (DN2), MDBT50Q_1.34 (D-)
- new net VBUS: C1.1, IC1.1 (IN), J2.A4 (VBUS_1), J2.B4 (VBUS_2), J8.1 (Pin_1), MDBT50Q_1.32 (VBUS)
- new net VIN_MEASURE: MDBT50Q_1.12 (P0.31/AIN7), R10.2, R9.1
- no-connect marks 0 -> 6
Other:
- note added: "3.3V Voltage Regulator"
- note added: "BLE / USB Mode Selector Switch"
- note added: "Battery Charging + Power Path"
- note added: "Fuel Gauge Voltage Divider"
- note added: "MCU"
- note added: "Normal Voltage mode"
- note added: "P0.13"
- note added: "P0.14"
- note added: "P0.15"
- note added: "P0.16"
- note added: "P0.17"
- note added: "P0.19"
- note added: "P0.20"
- note added: "P0.21"
- note added: "P0.22"
- note added: "P0.23"
- note added: "P0.30"
- note added: "P0.31"
- note added: "P1.00"
- note added: "P1.01"
- note added: "P1.10"
- note added: "Power Path Selection"
- note added: "Status LEDs"
- note added: "USB-C"
- moved on the sheet: D1, D10, D11, D12, D13, D14, D15, D16, D17, D18, D19, D2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

Commit message: initial keys layout
Parts:
- removed D2: 1N4148WS, Diode_SMD:D_SOD-323F, symbol Device:D_Small
- added D81: 1N4148WS, Diode_SMD:D_SOD-323F, symbol Device:D_Small
- SW10: value SW_Push -> A; footprint (none) -> Button_Switch_Keyboard:SW_Cherry_MX_1.00u_PCB
- SW11: value SW_Push -> Z; footprint (none) -> Button_Switch_Keyboard:SW_Cherry_MX_1.00u_PCB
- SW12: value SW_Push -> WIN; footprint (none) -> Button_Switch_Keyboard:SW_Cherry_MX_1.25u_PCB
- SW13: value SW_Push -> F1; footprint (none) -> Button_Switch_Keyboard:SW_Cherry_MX_1.00u_PCB
- SW14: value SW_Push -> 2; footprint (none) -> Button_Switch_Keyboard:SW_Cherry_MX_1.00u_PCB
- SW15: value SW_Push -> W; footprint (none) -> Button_Switch_Keyboard:SW_Cherry_MX_1.00u_PCB
- SW16: value SW_Push -> S; footprint (none) -> Button_Switch_Keyboard:SW_Cherry_MX_1.00u_PCB
- SW17: value SW_Push -> X; footprint (none) -> Button_Switch_Keyboard:SW_Cherry_MX_1.00u_PCB
- SW18: value SW_Push -> LALT; footprint (none) -> Button_Switch_Keyboard:SW_Cherry_MX_1.25u_PCB
- SW19: value SW_Push -> F2; footprint (none) -> Button_Switch_Keyboard:SW_Cherry_MX_1.00u_PCB
- SW2: value SW_Push -> ESC; footprint (none) -> Button_Switch_Keyboard:SW_Cherry_MX_1.00u_PCB
- SW20: value SW_Push -> 3; footprint (none) -> Button_Switch_Keyboard:SW_Cherry_MX_1.00u_PCB
- SW21: value SW_Push -> E; footprint (none) -> Button_Switch_Keyboard:SW_Cherry_MX_1.00u_PCB
- SW22: value SW_Push -> D; footprint (none) -> Button_Switch_Keyboard:SW_Cherry_MX_1.00u_PCB
- SW23: value SW_Push -> C; footprint (none) -> Button_Switch_Keyboard:SW_Cherry_MX_1.00u_PCB
- SW24: value SW_Push -> SPACE; footprint (none) -> Button_Switch_Keyboard:SW_Cherry_MX_6.25u_PCB
- SW25: value SW_Push -> F3; footprint (none) -> Button_Switch_Keyboard:SW_Cherry_MX_1.00u_PCB
- SW26: value SW_Push -> 4; footprint (none) -> Button_Switch_Keyboard:SW_Cherry_MX_1.00u_PCB
- SW27: value SW_Push -> R; footprint (none) -> Button_Switch_Keyboard:SW_Cherry_MX_1.00u_PCB
- SW28: value SW_Push -> F; footprint (none) -> Button_Switch_Keyboard:SW_Cherry_MX_1.00u_PCB
- SW29: value SW_Push -> V; footprint (none) -> Button_Switch_Keyboard:SW_Cherry_MX_1.00u_PCB
- SW3: value SW_Push -> TILDE; footprint (none) -> Button_Switch_Keyboard:SW_Cherry_MX_1.00u_PCB
- SW30: value SW_Push -> F4; footprint (none) -> Button_Switch_Keyboard:SW_Cherry_MX_1.00u_PCB
- SW31: value SW_Push -> 5; footprint (none) -> Button_Switch_Keyboard:SW_Cherry_MX_1.00u_PCB
- SW32: value SW_Push -> T; footprint (none) -> Button_Switch_Keyboard:SW_Cherry_MX_1.00u_PCB
- SW33: value SW_Push -> G; footprint (none) -> Button_Switch_Keyboard:SW_Cherry_MX_1.00u_PCB
- SW34: value SW_Push -> B; footprint (none) -> Button_Switch_Keyboard:SW_Cherry_MX_1.00u_PCB
- SW35: value SW_Push -> 6; footprint (none) -> Button_Switch_Keyboard:SW_Cherry_MX_1.00u_PCB
- SW36: value SW_Push -> Y; footprint (none) -> Button_Switch_Keyboard:SW_Cherry_MX_1.00u_PCB
- SW37: value SW_Push -> H; footprint (none) -> Button_Switch_Keyboard:SW_Cherry_MX_1.00u_PCB
- SW38: value SW_Push -> N; footprint (none) -> Button_Switch_Keyboard:SW_Cherry_MX_1.00u_PCB
- SW39: value SW_Push -> F5; footprint (none) -> Button_Switch_Keyboard:SW_Cherry_MX_1.00u_PCB
- SW4: value SW_Push -> TAB; footprint (none) -> Button_Switch_Keyboard:SW_Cherry_MX_1.50u_PCB
- SW40: value SW_Push -> 7; footprint (none) -> Button_Switch_Keyboard:SW_Cherry_MX_1.00u_PCB
- SW41: value SW_Push -> U; footprint (none) -> Button_Switch_Keyboard:SW_Cherry_MX_1.00u_PCB
- SW42: value SW_Push -> J; footprint (none) -> Button_Switch_Keyboard:SW_Cherry_MX_1.00u_PCB
- SW43: value SW_Push -> M; footprint (none) -> Button_Switch_Keyboard:SW_Cherry_MX_1.00u_PCB
- SW44: value SW_Push -> F6; footprint (none) -> Button_Switch_Keyboard:SW_Cherry_MX_1.00u_PCB
- SW45: value SW_Push -> 8; footprint (none) -> Button_Switch_Keyboard:SW_Cherry_MX_1.00u_PCB
- SW46: value SW_Push -> I; footprint (none) -> Button_Switch_Keyboard:SW_Cherry_MX_1.00u_PCB
- SW47: value SW_Push -> K; footprint (none) -> Button_Switch_Keyboard:SW_Cherry_MX_1.00u_PCB
- SW48: value SW_Push -> COMMA; footprint (none) -> Button_Switch_Keyboard:SW_Cherry_MX_1.00u_PCB
- SW49: value SW_Push -> RALT; footprint (none) -> Button_Switch_Keyboard:SW_Cherry_MX_1.25u_PCB
- SW5: value SW_Push -> CAPS; footprint (none) -> Button_Switch_Keyboard:SW_Cherry_MX_1.75u_PCB
- SW50: value SW_Push -> F7; footprint (none) -> Button_Switch_Keyboard:SW_Cherry_MX_1.00u_PCB
- SW51: value SW_Push -> 9; footprint (none) -> Button_Switch_Keyboard:SW_Cherry_MX_1.00u_PCB
- SW52: value SW_Push -> O; footprint (none) -> Button_Switch_Keyboard:SW_Cherry_MX_1.00u_PCB
- SW53: value SW_Push -> L; footprint (none) -> Button_Switch_Keyboard:SW_Cherry_MX_1.00u_PCB
- SW54: value SW_Push -> DOT; footprint (none) -> Button_Switch_Keyboard:SW_Cherry_MX_1.00u_PCB
- SW55: value SW_Push -> FN; footprint (none) -> Button_Switch_Keyboard:SW_Cherry_MX_1.25u_PCB
- SW56: value SW_Push -> F8; footprint (none) -> Button_Switch_Keyboard:SW_Cherry_MX_1.00u_PCB
- SW57: value SW_Push -> 0; footprint (none) -> Button_Switch_Keyboard:SW_Cherry_MX_1.00u_PCB
- SW58: value SW_Push -> P; footprint (none) -> Button_Switch_Keyboard:SW_Cherry_MX_1.00u_PCB
- SW59: value SW_Push -> SEMICOLON; footprint (none) -> Button_Switch_Keyboard:SW_Cherry_MX_1.00u_PCB
- SW6: value SW_Push -> LSHIFT; footprint (none) -> Button_Switch_Keyboard:SW_Cherry_MX_2.25u_PCB
- SW60: value SW_Push -> SLASH; footprint (none) -> Button_Switch_Keyboard:SW_Cherry_MX_1.00u_PCB
- SW61: value SW_Push -> MENU; footprint (none) -> Button_Switch_Keyboard:SW_Cherry_MX_1.25u_PCB
- SW62: value SW_Push -> MINUS; footprint (none) -> Button_Switch_Keyboard:SW_Cherry_MX_1.00u_PCB
- SW63: value SW_Push -> SQBOPEN; footprint (none) -> Button_Switch_Keyboard:SW_Cherry_MX_1.00u_PCB
- SW64: value SW_Push -> QUOTE; footprint (none) -> Button_Switch_Keyboard:SW_Cherry_MX_1.00u_PCB
- SW65: value SW_Push -> RSHIFT; footprint (none) -> Button_Switch_Keyboard:SW_Cherry_MX_2.75u_PCB
- SW66: value SW_Push -> RCTRL; footprint (none) -> Button_Switch_Keyboard:SW_Cherry_MX_1.25u_PCB
- SW67: value SW_Push -> F9; footprint (none) -> Button_Switch_Keyboard:SW_Cherry_MX_1.00u_PCB
- SW68: value SW_Push -> EQUAL; footprint (none) -> Button_Switch_Keyboard:SW_Cherry_MX_1.00u_PCB
- SW69: value SW_Push -> SQBCLOSE; footprint (none) -> Button_Switch_Keyboard:SW_Cherry_MX_1.00u_PCB
- SW7: value SW_Push -> LCTRL; footprint (none) -> Button_Switch_Keyboard:SW_Cherry_MX_1.25u_PCB
- SW70: value SW_Push -> ENTER; footprint (none) -> Button_Switch_Keyboard:SW_Cherry_MX_2.25u_PCB
- SW71: value SW_Push -> UP; footprint (none) -> Button_Switch_Keyboard:SW_Cherry_MX_1.00u_PCB
- SW72: value SW_Push -> LEFT; footprint (none) -> Button_Switch_Keyboard:SW_Cherry_MX_1.00u_PCB
- SW73: value SW_Push -> F10; footprint (none) -> Button_Switch_Keyboard:SW_Cherry_MX_1.00u_PCB
- SW74: value SW_Push -> BACKSPACE; footprint (none) -> Button_Switch_Keyboard:SW_Cherry_MX_2.00u_PCB
- SW75: value SW_Push -> FWDSLASH; footprint (none) -> Button_Switch_Keyboard:SW_Cherry_MX_1.50u_PCB
- SW76: value SW_Push -> DOWN; footprint (none) -> Button_Switch_Keyboard:SW_Cherry_MX_1.00u_PCB
- SW77: value SW_Push -> F11; footprint (none) -> Button_Switch_Keyboard:SW_Cherry_MX_1.00u_PCB
- SW78: value SW_Push -> PRTSCR; footprint (none) -> Button_Switch_Keyboard:SW_Cherry_MX_1.00u_PCB
- SW79: value SW_Push -> DEL; footprint (none) -> Button_Switch_Keyboard:SW_Cherry_MX_1.00u_PCB
- SW8: value SW_Push -> 1; footprint (none) -> Button_Switch_Keyboard:SW_Cherry_MX_1.00u_PCB
- SW80: value SW_Push -> RIGHT; footprint (none) -> Button_Switch_Keyboard:SW_Cherry_MX_1.00u_PCB
- SW81: value SW_Push -> F12; footprint (none) -> Button_Switch_Keyboard:SW_Cherry_MX_1.00u_PCB
- SW9: value SW_Push -> Q; footprint (none) -> Button_Switch_Keyboard:SW_Cherry_MX_1.00u_PCB
- renumbered D1 to D2
Connections:
- net COL_01: now also D2.2 (A), D8.2 (A), MDBT50Q_1.50 (P1.02), SW13.1, SW14.1, SW2.2, SW8.2; no longer SW12.1, SW2.1, SW22.1, SW32.1, SW42.1, SW52.1, SW62.1, SW72.1
- net COL_03: now also D13.2 (A), SW13.2, SW19.1; no longer SW14.1, SW24.1, SW34.1, SW4.1, SW44.1, SW54.1, SW64.1, SW74.1
- net COL_04: now also D19.2 (A), SW19.2; no longer SW15.1, SW35.1, SW45.1, SW5.1, SW55.1, SW65.1, SW75.1
- net COL_05: now also D25.2 (A), SW25.2, SW30.1; no longer SW16.1, SW26.1, SW36.1, SW46.1, SW56.1, SW6.1, SW66.1, SW76.1
- net COL_06: now also D30.2 (A), D35.2 (A), MDBT50Q_1.58 (P1.07), SW30.2, SW35.2, SW39.1, SW40.1; no longer SW17.1, SW27.1, SW37.1, SW47.1, SW57.1, SW67.1, SW7.1, SW77.1
- net COL_08: now also D39.2 (A), SW39.2, SW44.1; no longer SW19.1, SW29.1, SW39.1, SW49.1, SW59.1, SW69.1, SW79.1, SW9.1
- net COL_09: now also D44.2 (A), SW44.2; no longer SW10.1, SW20.1, SW30.1, SW40.1, SW60.1, SW70.1, SW80.1
- net COL_10: now also D50.2 (A), SW50.2, SW56.1; no longer SW11.1, SW21.1, SW31.1, SW41.1, SW51.1, SW61.1, SW71.1, SW81.1
- net ROW_01: now also SW2.1; no longer D17.1 (K), D2.1 (K), D25.1 (K), D33.1 (K), D41.1 (K), D49.1 (K), D57.1 (K), D65.1 (K), D73.1 (K), D9.1 (K)
- net ROW_02: now also SW3.1; no longer D10.1 (K), D18.1 (K), D26.1 (K), D34.1 (K), D42.1 (K), D50.1 (K), D58.1 (K), D66.1 (K), D74.1 (K)
- net ROW_03: now also SW4.1; no longer D11.1 (K), D19.1 (K), D27.1 (K), D3.1 (K), D35.1 (K), D43.1 (K), D51.1 (K), D59.1 (K), D67.1 (K), D75.1 (K)
- net ROW_04: now also SW5.1; no longer D12.1 (K), D20.1 (K), D28.1 (K), D36.1 (K), D4.1 (K), D44.1 (K), D52.1 (K), D60.1 (K), D68.1 (K), D76.1 (K)
- net ROW_05: now also SW6.1; no longer D13.1 (K), D21.1 (K), D29.1 (K), D37.1 (K), D45.1 (K), D5.1 (K), D53.1 (K), D61.1 (K), D69.1 (K), D77.1 (K)
- net ROW_06: now also SW7.1; no longer D14.1 (K), D22.1 (K), D30.1 (K), D38.1 (K), D46.1 (K), D54.1 (K), D6.1 (K), D62.1 (K), D70.1 (K), D78.1 (K)
- net at SW48.2: now also D47.1 (K), D48.2 (A), SW54.1; no longer D53.2 (A)
- net at D38.2 (A): now also D37.1 (K), SW38.2, SW43.1; no longer SW56.2
- net at SW64.2: now also D63.1 (K), D64.2 (A), SW70.1; no longer D23.2 (A)
- net at D59.2 (A): now also D58.1 (K), SW59.2, SW64.1; no longer SW29.2
- net at D7.2 (A): now also D6.1 (K), SW12.1, SW7.2; no longer SW62.2
- net at SW75.2: now also D74.1 (K), D75.2 (A), SW79.1; no longer D32.2 (A)
- net at D79.2 (A), SW71.2: now also D12.1 (K), D18.1 (K), D23.1 (K), D24.1 (K), D24.2 (A), D29.1 (K), D34.1 (K), D38.1 (K), D43.1 (K), D49.1 (K), D55.1 (K), D61.1 (K), D66.1 (K), D69.1 (K), D7.1 (K), D70.1 (K), D70.2 (A), D71.2 (A), D72.1 (K), D75.1 (K), D76.1 (K), D76.2 (A), D77.1 (K), D78.1 (K), D78.2 (A), D79.1 (K), D80.1 (K), D80.2 (A), SW24.2, SW49.1, SW70.2, SW76.2, SW78.2, SW79.2, SW80.1, SW80.2, D81.1 (K)
- net at D45.2 (A): now also D44.1 (K), SW45.2, SW51.1; no longer SW47.2
- net at SW61.2: now also D60.1 (K), D61.2 (A), SW66.1; no longer D78.2 (A)
- net at D47.2 (A): now also D46.1 (K), SW47.2, SW53.1; no longer SW67.2
- net at SW46.2: now also D45.1 (K), D46.2 (A), SW52.1; no longer D37.2 (A)
- net at D40.2 (A): now also D39.1 (K), SW40.2, SW45.1; no longer SW76.2
- net at SW34.2: now also D33.1 (K), D34.2 (A), SW38.1; no longer D20.2 (A)
- net at D52.2 (A): now also D51.1 (K), SW52.2, SW58.1; no longer SW38.2
- net at SW41.2: now also D40.1 (K), D41.2 (A), SW46.1; no longer D76.2 (A)
- net at D21.2 (A): now also D20.1 (K), SW21.2, SW27.1; no longer SW44.2
- net at SW57.2: now also D56.1 (K), D57.2 (A), SW62.1; no longer D46.2 (A)
- net at D18.2 (A): now also D17.1 (K), SW18.2, SW24.1; no longer SW14.2
- net at D29.2 (A): now also D28.1 (K), SW29.2, SW34.1; no longer SW45.2
- net at D63.2 (A): now also D62.1 (K), SW63.2, SW69.1; no longer SW69.2
- net at SW9.2: now also D8.1 (K), D9.2 (A), SW15.1; no longer D57.2 (A)
- net at D15.2 (A): now also D14.1 (K), SW15.2, SW21.1; no longer SW63.2
- net at SW51.2: now also D50.1 (K), D51.2 (A), SW57.1; no longer D77.2 (A)
- net at SW23.2: now also D22.1 (K), D23.2 (A), SW29.1; no longer D11.2 (A)
- net at SW31.2: now also D30.1 (K), D31.2 (A), SW35.1; no longer D75.2 (A)
- net at D68.2 (A): now also D67.1 (K), SW68.2, SW74.1; no longer SW40.2
- net at SW33.2: now also D32.1 (K), D33.2 (A), SW37.1; no longer D12.2 (A)
- net at SW3.2: now also D2.1 (K), D3.2 (A), SW8.1; no longer D9.2 (A)
- net at SW6.2: now also D5.1 (K), D6.2 (A), SW11.1; no longer D33.2 (A)
- net at SW58.2: now also D57.1 (K), D58.2 (A), SW63.1; no longer D54.2 (A)
- net at SW12.2: now also D11.1 (K), D12.2 (A), SW18.1
- net at SW26.2: now also D25.1 (K), D26.2 (A), SW31.1; no longer D35.2 (A)
- net at D69.2 (A): now also D68.1 (K), SW69.2, SW75.1; no longer SW50.2
- net at SW49.2: now also D48.1 (K), D49.2 (A), SW55.1; no longer D61.2 (A)
- net at D27.2 (A): now also D26.1 (K), SW27.2, SW32.1; no longer SW25.2
- net at SW60.2: now also D59.1 (K), D60.2 (A), SW65.1; no longer D70.2 (A)
- net at D43.2 (A): now also D42.1 (K), SW43.2, SW48.1; no longer SW27.2
- net at SW5.2: now also D4.1 (K), D5.2 (A), SW10.1; no longer D25.2 (A)
- net at SW17.2: now also D16.1 (K), D17.2 (A), SW23.1; no longer D42.2 (A)
- net at SW22.2: now also D21.1 (K), D22.2 (A), SW28.1; no longer D3.2 (A)
- net at D4.2 (A): now also D3.1 (K), SW4.2, SW9.1; no longer SW32.2
- net COL_13: now reaches D67.2 (A)
- net COL_13: now also MDBT50Q_1.6 (P1.13), SW67.2, SW73.1; no longer SW30.2
- net at SW54.2: now also D53.1 (K), D54.2 (A), SW60.1; no longer D22.2 (A)
- net at SW66.2: now also D65.1 (K), D66.2 (A), SW72.1; no longer D39.2 (A)
- net at SW53.2: now also D52.1 (K), D53.2 (A), SW59.1; no longer D14.2 (A)
- net at D72.2 (A): now also D71.1 (K), SW72.2, SW76.1; no longer SW80.2
- net at D16.2 (A): now also D15.1 (K), SW16.2, SW22.1; no longer SW73.2
- net at D10.2 (A): now also D9.1 (K), SW10.2, SW16.1; no longer SW13.2
- net COL_11: now reaches MDBT50Q_1.4 (P1.11)
- net COL_11: now also D56.2 (A), D62.2 (A), MDBT50Q_1.5 (P1.12), SW56.2, SW62.2, SW67.1, SW68.1
- net COL_14: now reaches MDBT50Q_1.7 (P1.14)
- net COL_14: now also D73.2 (A), SW73.2, SW77.1
- net COL_15: now reaches MDBT50Q_1.8 (P1.15)
- net COL_15: now also D77.2 (A), SW77.2, SW81.1
- net COL_16: now reaches MDBT50Q_1.9 (P0.03/AIN1)
- net COL_16: now also SW81.2, D81.2 (A)
- net at D28.2 (A): now also D27.1 (K), SW28.2, SW33.1; no longer SW35.2
- net at SW20.2: now also D19.1 (K), D20.2 (A), SW26.1; no longer D66.2 (A)
- net at D74.2 (A): now also D73.1 (K), SW74.2, SW78.1; no longer SW21.2
- net at D65.2 (A): now also D64.1 (K), SW65.2, SW71.1; no longer SW10.2
- net at SW11.2: now also D10.1 (K), D11.2 (A), SW17.1; no longer D73.2 (A)
- net at SW37.2: now also D36.1 (K), D37.2 (A), SW42.1; no longer D44.2 (A)
- net at SW42.2: now also D41.1 (K), D42.2 (A), SW47.1; no longer D5.2 (A)
- net at D36.2 (A), SW36.2: now also D35.1 (K), SW41.1
- net at D55.2 (A): now also D54.1 (K), SW55.2, SW61.1; no longer SW68.2
- removed net COL_02: MDBT50Q_1.50 (P1.02), SW13.1, SW23.1, SW3.1, SW33.1, SW43.1, SW53.1, SW63.1, SW73.1
- removed net COL_07: MDBT50Q_1.58 (P1.07), SW18.1, SW28.1, SW38.1, SW48.1, SW58.1, SW68.1, SW78.1, SW8.1
- removed net ROW_07: D15.1 (K), D23.1 (K), D31.1 (K), D39.1 (K), D47.1 (K), D55.1 (K), D63.1 (K), D7.1 (K), D71.1 (K), D79.1 (K), MDBT50Q_1.10 (P0.29/AIN5)
- removed net ROW_08: D16.1 (K), D24.1 (K), D32.1 (K), D40.1 (K), D48.1 (K), D56.1 (K), D64.1 (K), D72.1 (K), D8.1 (K), D80.1 (K), MDBT50Q_1.14 (P0.30/AIN6)
- new net: D31.1 (K), D32.2 (A), SW32.2, SW36.1
- new net: D13.1 (K), D14.2 (A), SW14.2, SW20.1
Other:
- note added: "P0.03"
- note added: "P0.28"
- note added: "P1.15"
- note added: "Total GPIO = 22 ROW01-06 COL01-16"
- note removed: "P0.30"
- note removed: "P1.10"
- note removed: "Total GPIO = 18 ROW01-08 COL01-10"
- moved on the sheet: C3, C4, C5, D2, IC2, J7, L2, R10, R9, SW2

Commit message: layout rev1
Parts:
- removed D71, D72, D76, D78, D79, D80: 1N4148WS, Diode_SMD:D_SOD-323F, symbol Device:D_Small
- removed J2: UJ20-C-H-G-MSMT-4B-P16-TR, usbc_lion:UJ20CHGMSMT4BP16TR, symbol UJ20-C-H-G-MSMT-4B-P16-TR:UJ20-C-H-G-MSMT-4B-P16-TR
- removed J3: Battery, Connector_PinHeader_2.54mm:PinHeader_1x02_P2.54mm_Vertical, symbol Connector_Generic:Conn_01x02
- removed SW71: UP, Button_Switch_Keyboard:SW_Cherry_MX_1.00u_PCB, symbol Switch:SW_Push
- removed SW72: LEFT, Button_Switch_Keyboard:SW_Cherry_MX_1.00u_PCB, symbol Switch:SW_Push
- removed SW76: DOWN, Button_Switch_Keyboard:SW_Cherry_MX_1.00u_PCB, symbol Switch:SW_Push
- removed SW78: PRTSCR, Button_Switch_Keyboard:SW_Cherry_MX_1.00u_PCB, symbol Switch:SW_Push
- removed SW79: DEL, Button_Switch_Keyboard:SW_Cherry_MX_1.00u_PCB, symbol Switch:SW_Push
- removed SW80: RIGHT, Button_Switch_Keyboard:SW_Cherry_MX_1.00u_PCB, symbol Switch:SW_Push
- added J2: USB4216-03-A, USB421603A, symbol USB4216-03-A:USB4216-03-A
- J8: footprint Connector_PinHeader_2.54mm:PinHeader_1x03_P2.54mm_Vertical -> Connector_PinHeader_2.54mm:PinHeader_1x04_P2.54mm_Vertical; symbol Connector_Generic:Conn_01x03 -> Connector_Generic:Conn_01x04
Connections:
- net COL_15: no longer SW81.1
- net GND: now also J8.4 (Pin_4), J2.A1 (GND_1), J2.B1 (GND_2), J2.G1 (GND_3), J2.G2 (GND_4), J2.G3 (GND_5), J2.G4 (GND_6)
- net USB_CC1: now also J2.A5 (CC1)
- net USB_CC2: now also J2.B5 (CC2)
- net USB_D+: now also J2.A6 (DP1), J2.B6 (DP2)
- net USB_D-: now also J2.A7 (DN1), J2.B7 (DN2)
- net VBUS: now also J2.A4 (VBUS_1), J2.B4 (VBUS_2)
- net at D12.1 (K), D18.1 (K), D23.1 (K)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: now also D64.1 (K), D65.1 (K), D65.2 (A), D66.2 (A), D74.1 (K), D75.2 (A), SW65.2, SW66.2, SW75.2; no longer D77.1 (K)
- net at D73.1 (K), D74.2 (A), SW74.2: now also SW81.1
- net COL_16: no longer names the net of D81.2 (A), SW81.2
- net COL_16: now also D77.1 (K); no longer MDBT50Q_1.9 (P0.03/AIN1)
- no-connect marks 6 -> 2
Other:
- note removed: "P0.03"
- moved on the sheet: D81, SW81

Commit message: schematics update + routing progress
Connections:
- net COL_01: now also SW2.1, SW3.1, SW4.1, SW5.1, SW6.1, SW7.1; no longer D2.2 (A), D8.2 (A), MDBT50Q_1.50 (P1.02), SW13.1, SW14.1, SW2.2, SW8.2
- net COL_03: now also SW13.1, SW14.1, SW15.1, SW16.1, SW17.1, SW18.1; no longer D13.2 (A), SW13.2, SW19.1
- net COL_04: now also SW19.1, SW20.1, SW21.1, SW22.1, SW23.1, SW24.1; no longer D19.2 (A), SW19.2, SW25.1
- net COL_05: now also SW25.1, SW26.1, SW27.1, SW28.1, SW29.1; no longer D25.2 (A), SW25.2, SW30.1
- net COL_06: now also SW30.1, SW31.1, SW32.1, SW33.1, SW34.1; no longer D30.2 (A), D35.2 (A), MDBT50Q_1.58 (P1.07), SW30.2, SW35.2, SW39.1, SW40.1
- net COL_08: now also SW39.1, SW40.1, SW41.1, SW42.1, SW43.1; no longer D39.2 (A), SW39.2, SW44.1
- net COL_09: now also SW44.1, SW45.1, SW46.1, SW47.1, SW48.1, SW49.1; no longer D44.2 (A), SW44.2, SW50.1
- net COL_10: now also SW50.1, SW51.1, SW52.1, SW53.1, SW54.1, SW55.1; no longer D50.2 (A), SW50.2, SW56.1
- net COL_11: now also SW56.1, SW57.1, SW58.1, SW59.1, SW60.1, SW61.1; no longer D56.2 (A), D62.2 (A), MDBT50Q_1.5 (P1.12), SW56.2, SW62.2, SW67.1, SW68.1
- net COL_13: now also SW67.1, SW68.1, SW69.1, SW70.1; no longer D67.2 (A), SW67.2, SW73.1
- net COL_14: now also SW73.1, SW74.1, SW75.1; no longer D73.2 (A), SW73.2, SW77.1
- net COL_15: now also SW77.1, SW81.1; no longer D77.2 (A), SW77.2
- net ROW_01: now also D13.1 (K), D19.1 (K), D2.1 (K), D25.1 (K), D30.1 (K), D39.1 (K), D44.1 (K), D50.1 (K), D56.1 (K), D67.1 (K), D73.1 (K), D77.1 (K); no longer SW2.1
- net ROW_02: now also D14.1 (K), D20.1 (K), D26.1 (K), D3.1 (K), D31.1 (K), D35.1 (K), D40.1 (K), D45.1 (K), D51.1 (K), D57.1 (K), D62.1 (K), D68.1 (K), D74.1 (K), D8.1 (K), D81.1 (K); no longer SW3.1
- net ROW_03: now also D15.1 (K), D21.1 (K), D27.1 (K), D32.1 (K), D36.1 (K), D4.1 (K), D41.1 (K), D46.1 (K), D52.1 (K), D58.1 (K), D63.1 (K), D69.1 (K), D75.1 (K), D9.1 (K); no longer SW4.1
- net ROW_04: now also D10.1 (K), D16.1 (K), D22.1 (K), D28.1 (K), D33.1 (K), D37.1 (K), D42.1 (K), D47.1 (K), D5.1 (K), D53.1 (K), D59.1 (K), D64.1 (K), D70.1 (K); no longer SW5.1
- net ROW_05: now also D11.1 (K), D17.1 (K), D23.1 (K), D29.1 (K), D34.1 (K), D38.1 (K), D43.1 (K), D48.1 (K), D54.1 (K), D6.1 (K), D60.1 (K), D65.1 (K); no longer SW6.1
- net ROW_06: now also D12.1 (K), D18.1 (K), D24.1 (K), D49.1 (K), D55.1 (K), D61.1 (K), D66.1 (K), D7.1 (K); no longer SW7.1
- net at D17.2 (A), SW17.2: no longer D16.1 (K), SW23.1
- net at D16.2 (A), SW16.2: no longer D15.1 (K), SW22.1
- net at D59.2 (A), SW59.2: no longer D58.1 (K), SW64.1
- net at D64.2 (A), SW64.2: no longer D63.1 (K), SW70.1
- net at D68.2 (A), SW68.2: no longer D67.1 (K), SW74.1
- net at D74.2 (A), SW74.2: no longer D73.1 (K), SW81.1
- net at D61.2 (A), SW61.2: no longer D60.1 (K), SW66.1
- net at D60.2 (A), SW60.2: no longer D59.1 (K), SW65.1
- net at D10.2 (A), SW10.2: no longer D9.1 (K), SW16.1
- net at D9.2 (A), SW9.2: no longer D8.1 (K), SW15.1
- net at D40.2 (A), SW40.2: no longer D39.1 (K), SW45.1
- net at D45.2 (A), SW45.2: no longer D44.1 (K), SW51.1
- net at D34.2 (A), SW34.2: no longer D33.1 (K), SW38.1
- net at D5.2 (A), SW5.2: no longer D4.1 (K), SW10.1
- net at D4.2 (A), SW4.2: no longer D3.1 (K), SW9.1
- net at D63.2 (A), SW63.2: no longer D62.1 (K), SW69.1
- net at D69.2 (A), SW69.2: no longer D68.1 (K), SW75.1
- net at D49.2 (A), SW49.2: no longer D48.1 (K), SW55.1
- net at D18.2 (A), SW18.2: no longer D17.1 (K), SW24.1
- net at D47.2 (A), SW47.2: no longer D46.1 (K), SW53.1
- net at D46.2 (A), SW46.2: no longer D45.1 (K), SW52.1
- net at D58.2 (A), SW58.2: no longer D57.1 (K), SW63.1
- net at D57.2 (A), SW57.2: no longer D56.1 (K), SW62.1
- net at D48.2 (A), SW48.2: no longer D47.1 (K), SW54.1
- net at D23.2 (A), SW23.2: no longer D22.1 (K), SW29.1
- net at D36.2 (A), SW36.2: no longer D35.1 (K), SW41.1
- net at D41.2 (A), SW41.2: no longer D40.1 (K), SW46.1
- net at D11.2 (A), SW11.2: no longer D10.1 (K), SW17.1
- net at D7.2 (A), SW7.2: no longer D6.1 (K), SW12.1
- net at D6.2 (A), SW6.2: no longer D5.1 (K), SW11.1
- net at D38.2 (A), SW38.2: no longer D37.1 (K), SW43.1
- net at D55.2 (A), SW55.2: no longer D54.1 (K), SW61.1
- net at D15.2 (A), SW15.2: no longer D14.1 (K), SW21.1
- net at D43.2 (A), SW43.2: no longer D42.1 (K), SW48.1
- net at D27.2 (A), SW27.2: no longer D26.1 (K), SW32.1
- net at D32.2 (A), SW32.2: no longer D31.1 (K), SW36.1
- net at D37.2 (A), SW37.2: no longer D36.1 (K), SW42.1
- net at D42.2 (A), SW42.2: no longer D41.1 (K), SW47.1
- net at D22.2 (A), SW22.2: no longer D21.1 (K), SW28.1
- net at D26.2 (A), SW26.2: no longer D25.1 (K), SW31.1
- net at D33.2 (A), SW33.2: no longer D32.1 (K), SW37.1
- net at D31.2 (A), SW31.2: no longer D30.1 (K), SW35.1
- net at D28.2 (A), SW28.2: no longer D27.1 (K), SW33.1
- net at D53.2 (A), SW53.2: no longer D52.1 (K), SW59.1
- net at D52.2 (A), SW52.2: no longer D51.1 (K), SW58.1
- net at D21.2 (A), SW21.2: no longer D20.1 (K), SW27.1
- net at D20.2 (A), SW20.2: no longer D19.1 (K), SW26.1
- net at D54.2 (A), SW54.2: no longer D53.1 (K), SW60.1
- net at D81.2 (A), SW81.2: no longer D77.1 (K)
- net at D3.2 (A), SW3.2: no longer D2.1 (K), SW8.1
- net at D14.2 (A), SW14.2: no longer D13.1 (K), SW20.1
- net at D51.2 (A), SW51.2: no longer D50.1 (K), SW57.1
- net at D29.2 (A), SW29.2: no longer D28.1 (K), SW34.1
- net at D12.2 (A), SW12.2: no longer D11.1 (K), SW18.1
- new net: D66.2 (A), SW66.2
- new net: D19.2 (A), SW19.2
- new net: D73.2 (A), SW73.2
- new net: D65.2 (A), SW65.2
- new net: D75.2 (A), SW75.2
- new net: D24.2 (A), SW24.2
- new net: D77.2 (A), SW77.2
- new net: D35.2 (A), SW35.2
- new net: D62.2 (A), SW62.2
- new net: D25.2 (A), SW25.2
- new net: D30.2 (A), SW30.2
- new net: D13.2 (A), SW13.2
- new net: D44.2 (A), SW44.2
- new net: D2.2 (A), SW2.2
- new net: D50.2 (A), SW50.2
- new net: D39.2 (A), SW39.2
- new net: D56.2 (A), SW56.2
- new net: D67.2 (A), SW67.2
- new net: D8.2 (A), SW8.2
- new net: D70.2 (A), SW70.2
- new net COL_02: MDBT50Q_1.50 (P1.02), SW10.1, SW11.1, SW12.1, SW8.1, SW9.1
- new net COL_07: MDBT50Q_1.58 (P1.07), SW35.1, SW36.1, SW37.1, SW38.1
- new net COL_12: MDBT50Q_1.5 (P1.12), SW62.1, SW63.1, SW64.1, SW65.1, SW66.1
Other:
- moved on the sheet: D10, D11, D12, D13, D14, D15, D16, D17, D18, D19, D2, D20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

Commit message: routing almost finished
Parts:
- added J3: ProgConn, Connector_PinHeader_2.54mm:PinHeader_1x04_P2.54mm_Vertical, symbol Connector_Generic:Conn_01x04
Connections:
- net +3.3V: now also J3.4 (Pin_4)
- net COL_01: now also MDBT50Q_1.13 (P0.28/AIN4); no longer MDBT50Q_1.61 (P1.01)
- net COL_02: now also MDBT50Q_1.14 (P0.30/AIN6); no longer MDBT50Q_1.50 (P1.02)
- net COL_03: now also MDBT50Q_1.16 (P0.27); no longer MDBT50Q_1.60 (P1.03)
- net COL_04: now also MDBT50Q_1.17 (P0.00/XL1); no longer MDBT50Q_1.56 (P1.04)
- net COL_05: now also MDBT50Q_1.18 (P0.01/XL2); no longer MDBT50Q_1.59 (P1.05)
- net COL_06: now also MDBT50Q_1.19 (P0.26); no longer MDBT50Q_1.57 (P1.06)
- net COL_07: now also MDBT50Q_1.20 (P0.04/AIN2); no longer MDBT50Q_1.58 (P1.07)
- net COL_08: now also MDBT50Q_1.21 (P0.05/AIN3); no longer MDBT50Q_1.25 (P1.08)
- net COL_09: now also MDBT50Q_1.22 (P0.06); no longer MDBT50Q_1.26 (P1.09)
- net COL_10: now also MDBT50Q_1.23 (P0.07); no longer MDBT50Q_1.3 (P1.10)
- net COL_11: now also MDBT50Q_1.24 (P0.08); no longer MDBT50Q_1.4 (P1.11)
- net COL_12: now also MDBT50Q_1.25 (P1.08); no longer MDBT50Q_1.5 (P1.12)
- net COL_13: now also MDBT50Q_1.26 (P1.09); no longer MDBT50Q_1.6 (P1.13)
- net COL_14: now also MDBT50Q_1.27 (P0.11); no longer MDBT50Q_1.7 (P1.14)
- net COL_15: now also MDBT50Q_1.29 (P0.12); no longer MDBT50Q_1.8 (P1.15)
- net GND: now also J3.3 (Pin_3)
- net MCU_SWDCLK: now also J3.2 (Pin_2)
- net MCU_SWDIO: now also J3.1 (Pin_1)
- net ROW_01: now also MDBT50Q_1.4 (P1.11); no longer MDBT50Q_1.45 (P0.23)
- net ROW_02: now also MDBT50Q_1.5 (P1.12); no longer MDBT50Q_1.48 (P0.24)
- net ROW_03: now also MDBT50Q_1.6 (P1.13); no longer MDBT50Q_1.49 (P0.25)
- net ROW_04: now also MDBT50Q_1.7 (P1.14); no longer MDBT50Q_1.19 (P0.26)
- net ROW_05: now also MDBT50Q_1.8 (P1.15); no longer MDBT50Q_1.16 (P0.27)
- net ROW_06: now also MDBT50Q_1.9 (P0.03/AIN1); no longer MDBT50Q_1.13 (P0.28/AIN4)
Other:
- note removed: "P0.23"
- note removed: "P0.28"
- note removed: "P1.01"
- note removed: "P1.15"
