File: PCB/Original/K-0.kicad_sch (KiCad schematic)
At the start: 177 parts, among them IC1 BQ24040DSQR, IC2 TPS63031DSKR, J1 Display, J2 USB4216-03-A, J3 ProgConn, J4 PG_LED, J5 CHRG_LED, J6 POWER_LED, J7 Mode Selector, J8 Mode Selector, J9 LED_STRIP, SW1 RotaryEncoder_Switch, SW10 A, SW11 Z, SW12 WIN, SW13 F1, SW14 2, SW15 W, SW16 S, SW17 X, SW18 LALT, SW19 F2, SW2 ESC, SW20 3, SW21 E, SW22 D, SW23 C, SW24 SPACE, SW25 F3, SW26 4, SW27 R, SW28 F, SW29 V, SW3 TILDE, SW30 F4, SW31 5, SW32 T, SW33 G, SW34 B, SW35 6, SW36 Y, SW37 H, SW38 N, SW39 F5, SW4 TAB, SW40 7, SW41 U, SW42 J, SW43 M, SW44 F6, SW45 8, SW46 I, SW47 K, SW48 COMMA, SW49 RALT, SW5 CAPS, SW50 F7, SW51 9, SW52 O, SW53 L, SW54 DOT, SW55 FN, SW56 F8, SW57 0, SW58 P, SW59 SEMICOLON, SW6 LSHIFT, SW60 SLASH, SW61 MENU, SW62 MINUS, SW63 SQBOPEN, SW64 QUOTE, SW65 RSHIFT, SW66 RCTRL, SW67 F9, SW68 EQUAL, SW69 SQBCLOSE, SW7 LCTRL, SW70 ENTER, SW73 F10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

Commit message: v2 init
Parts:
- J1: CAD Model Link (none) -> https://grabcad.com/library/adafruit-neopixel-stick-8-neopi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; now left out of the parts list
- J3, J4, J5, J6, J7, J8, J9, R10, R3, R4, R5, R6, R7, R8, R9, SW1, SW10, SW11, SW12, SW13, SW14, SW15, SW16, SW17, SW18, SW19, SW2, SW20, SW21, SW22, SW23, SW24, SW25, SW26, SW27, SW28, SW29, SW3, SW30, SW31, SW32, SW33, SW34, SW35, SW36, SW37, SW38, SW39, SW4, SW40, SW41, SW42, SW43, SW44, SW45, SW46, SW47, SW48, SW49, SW5, SW50, SW51, SW52, SW53, SW54, SW55, SW56, SW57, SW58, SW59, SW6, SW60, SW61, SW62, SW63, SW64, SW65, SW66, SW67, SW68, SW69, SW7, SW70, SW73, SW74, SW75, SW77, SW8, SW81, SW9: now left out of the parts list
