File: PCB/daughter_board/daughter_board.kicad_pcb (KiCad board)
At the start: 4 copper layers, 291.2 x 130.9 mm, 180 parts, among them IC1 BQ24040DSQR, IC2 TPS63031DSKR, J1 Display, J10 key_board_conn, J11 main_board_conn, J2 USB4216-03-A, J3 ProgConn, J4 PG_LED, J5 CHRG_LED, J6 POWER_LED, J7 Mode Selector, J8 Mode Selector, J9 LED_STRIP, SW1 RotaryEncoder_Switch, SW10 A, SW11 Z, SW12 WIN, SW13 F1, SW14 2, SW15 W, SW16 S, SW17 X, SW18 LALT, SW19 F2, SW2 ESC, SW20 3, SW21 E, SW22 D, SW23 C, SW24 SPACE, SW25 F3, SW26 4, SW27 R, SW28 F, SW29 V, SW3 TILDE, SW30 F4, SW31 5, SW32 T, SW33 G, SW34 B, SW35 6, SW36 Y, SW37 H, SW38 N, SW39 F5, SW4 TAB, SW40 7, SW41 U, SW42 J, SW43 M, SW44 F6, SW45 8, SW46 I, SW47 K, SW48 COMMA, SW49 RALT, SW5 CAPS, SW50 F7, SW51 9, SW52 O, SW53 L, SW54 DOT, SW55 FN, SW56 F8, SW57 0, SW58 P, SW59 SEMICOLON, SW6 LSHIFT, SW60 SLASH, SW61 MENU, SW62 MINUS, SW63 SQBOPEN, SW64 QUOTE, SW65 RSHIFT, SW66 RCTRL, SW67 F9, SW68 EQUAL, SW69 SQBCLOSE, SW7 LCTRL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

Commit message: added teardrops on daughter board
Parts:
- removed C1, C2: 1uF, Capacitor_SMD:C_0402_1005Metric
- removed C3, C4: 10uF, Capacitor_SMD:C_0402_1005Metric
- removed C5: 0.1uF, Capacitor_SMD:C_0402_1005Metric
- removed IC1: BQ24040DSQR, BQ24040DSQR-lion:SON40P200X200X80-11N
- removed IC2: TPS63031DSKR, TPS63031DSKR-lion:SON50P250X250X80-11N-D
- removed J1: Display, Connector_PinHeader_2.54mm:PinHeader_1x08_P2.54mm_Vertical
- removed J11: main_board_conn, Connector_PinHeader_2.54mm:PinHeader_1x26_P2.54mm_Vertical
- removed J2: USB4216-03-A, usbc-lion:USB421603A
- removed J3: ProgConn, Connector_PinHeader_2.54mm:PinHeader_1x04_P2.54mm_Vertical
- removed J4: PG_LED, Connector_PinHeader_2.54mm:PinHeader_1x02_P2.54mm_Vertical
- removed J5: CHRG_LED, Connector_PinHeader_2.54mm:PinHeader_1x02_P2.54mm_Vertical
- removed J6: POWER_LED, Connector_PinHeader_2.54mm:PinHeader_1x02_P2.54mm_Vertical
- removed J7: Mode Selector, Connector_PinHeader_2.54mm:PinHeader_1x03_P2.54mm_Vertical
- removed J8: Mode Selector, Connector_PinHeader_2.54mm:PinHeader_1x04_P2.54mm_Vertical
- removed J9: LED_STRIP, Connector_PinHeader_2.54mm:PinHeader_1x03_P2.54mm_Vertical
- removed L2: LPS3015-222MRC, LPS3015-222MRC:IND_LPS3015-222MRC
- removed MDBT50Q_1: MDBT50Q_1, RF_Module:Raytac_MDBT50Q
- removed R1, R2: 5.1k, Resistor_SMD:R_0402_1005Metric
- removed R10: 400k, Connector_PinHeader_2.54mm:PinHeader_1x02_P2.54mm_Vertical
- removed R3: 1k, Connector_PinHeader_2.54mm:PinHeader_1x02_P2.54mm_Vertical
- removed R4: 2k, Connector_PinHeader_2.54mm:PinHeader_1x02_P2.54mm_Vertical
- removed R5: 10k, Connector_PinHeader_2.54mm:PinHeader_1x02_P2.54mm_Vertical
- removed R6, R7, R8: 330, Connector_PinHeader_2.54mm:PinHeader_1x02_P2.54mm_Vertical
- removed R9: 300k, Connector_PinHeader_2.54mm:PinHeader_1x02_P2.54mm_Vertical
Routing:
- net GND: track 46.5 -> 6.45 mm, vias 416 -> 372
- net /Display_CS: track 34.8 -> 0.00 mm, vias 2 -> 0
- net /Display_SCLK: track 33.6 -> 0.00 mm
- net /Display_MOSI: track 30.9 -> 0.00 mm
- net /Display_RES: track 29.9 -> 0.00 mm, vias 2 -> 0
- net /Display_DC: track 22.5 -> 0.00 mm
- net +3.3V: track 22.1 -> 0.00 mm, vias 1 -> 0
- net /MCU_SWDIO: track 21.0 -> 0.00 mm
- net /Display_BLK: track 20.1 -> 0.00 mm
- net Net-(IC1-PRETERM): track 19.4 -> 0.00 mm
- net /MCU_SWDCLK: track 18.3 -> 0.00 mm
- net Net-(IC1-ISET): track 13.4 -> 0.00 mm
- net /CHRG_LED: track 12.9 -> 0.00 mm
- net Net-(IC1-TS): track 12.5 -> 0.00 mm
- net /MODE_SEL_PIN: track 10.9 -> 0.00 mm, vias 1 -> 0
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Other:
- copper layers 4 -> 2
- board text removed: "(NOT ON PCB, WILL BE RAISED UP)"
- board text removed: "+"
- board text removed: "-"
- board text removed: "3V3"
- board text removed: "3V3/GND/SWDCLK/SWDIO"
- board text removed: "3v3"
- board text removed: "BAT"
- board text removed: "BLK"
- board text removed: "D"
- board text removed: "DISPLAY_CONN"
- board text removed: "DISPLAY_MODULE"
- board text removed: "MODE_SEL_SW"
- board text removed: "POWER_SEL_SWITCH"
- board text removed: "Programmer"

Commit message: updated daughter board
Routing:
- net GND: vias 372 -> 374

Commit message: pcb finish rev2
Parts:
- added G***: LOGO, LOGO, F.Cu at (292.1, 243.2)
- added G***: LOGO, LOGO, F.Cu at (301.2, 241.6)
- added G***: LOGO, LOGO, F.Cu at (279.4, 231.4)
- added G***: LOGO, LOGO, F.Cu at (323.2, 243.8)
- added G***: LOGO, LOGO, F.Cu at (249.1, 243.5)
- added G***: LOGO, LOGO, F.Cu at (324.4, 237.7)
- added G***: LOGO, LOGO, F.Cu at (277.9, 243.0)
- added G***: LOGO, LOGO, F.Cu at (273.4, 236.9)
- added G***: LOGO, LOGO, F.Cu at (319.4, 242.8)
- added G***: LOGO, LOGO, F.Cu at (323.6, 229.8)
- added G***: LOGO, LOGO, F.Cu at (307.1, 229.8)
- added G***: LOGO, LOGO, F.Cu at (295.8, 239.3)
- added G***: LOGO, LOGO, F.Cu at (309.5, 240.1)
- added G***: LOGO, LOGO, F.Cu at (315.3, 234.7)
- added G***: LOGO, LOGO, F.Cu at (202.7, 243.3)
- added G***: LOGO, LOGO, F.Cu at (205.6, 229.9)
- added G***: LOGO, LOGO, F.Cu at (299.6, 234.6)
- added G***: LOGO, LOGO, F.Cu at (285.0, 237.7)
- added G***: LOGO, LOGO, F.Cu at (301.6, 230.1)
- added G***: LOGO, LOGO, F.Cu at (279.1, 237.5)
- added G***: LOGO, LOGO, F.Cu at (291.7, 231.3)
- D10, D11, D12, D13, D14, D15, D16, D17, D18, D19, D2, D20, D21, D22, D23, D24, D25, D26, D27, D28, D29, D3, D30, D31, D32, D33, D34, D35, D36, D37, D38, D39, D4, D40, D41, D42, D43, D44, D45, D46, D47, D48, D49, D5, D50, D51, D52, D53, D54, D55, D56, D57, D58, D59, D6, D60, D61, D62, D63, D64, D65, D66, D67, D68, D69, D7, D70, D73, D74, D75, D77, D8, D81, D9: value 1N4148WS -> 1N4148TA; footprint Diode_SMD:D_SOD-323F -> Diode_THT:D_DO-35_SOD27_P7.62mm_Horizontal
- moved G*** 1.10 mm to (155.5, 134.4)
Routing:
- net /ROW_06: track 442.4 -> 520.5 mm, vias 1 -> 3
- net /ROW_05: track 385.3 -> 365.9 mm, vias 1 -> 3
- net GND: track 6.45 -> 22.0 mm, vias 374 -> 378
- net /ROW_03: track 350.6 -> 339.9 mm, vias 1 -> 2
- net /ROW_04: track 365.5 -> 357.2 mm, vias 1 -> 2
- net /ROW_02: track 360.0 -> 366.1 mm, vias 1 -> 0
- net /ROW_01: track 296.2 -> 299.0 mm, vias 1 -> 0
- net /COL_11: track 153.1 -> 150.3 mm
- net /COL_03: track 258.8 -> 260.7 mm
- net /COL_02: track 274.0 -> 275.6 mm
- net Net-(D52-A): track 11.8 -> 13.2 mm
- net Net-(D77-A): track 11.8 -> 13.2 mm
- net Net-(D61-A): track 11.8 -> 13.2 mm
- net Net-(D24-A): track 11.8 -> 13.2 mm
- net Net-(D64-A): track 11.8 -> 13.2 mm
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Other:
- outline, holes or cut-outs redrawn
- board text added: "3"
- board text added: "welcome, stranger."
- board text added: "you have discovered the area beaneath space!"
