File: PCB/daughter_board/daughter_board.kicad_sch (KiCad schematic)
At the start: 177 parts, among them IC1 BQ24040DSQR, IC2 TPS63031DSKR, J1 Display, J2 USB4216-03-A, J3 ProgConn, J4 PG_LED, J5 CHRG_LED, J6 POWER_LED, J7 Mode Selector, J8 Mode Selector, J9 LED_STRIP, SW1 RotaryEncoder_Switch, SW10 A, SW11 Z, SW12 WIN, SW13 F1, SW14 2, SW15 W, SW16 S, SW17 X, SW18 LALT, SW19 F2, SW2 ESC, SW20 3, SW21 E, SW22 D, SW23 C, SW24 SPACE, SW25 F3, SW26 4, SW27 R, SW28 F, SW29 V, SW3 TILDE, SW30 F4, SW31 5, SW32 T, SW33 G, SW34 B, SW35 6, SW36 Y, SW37 H, SW38 N, SW39 F5, SW4 TAB, SW40 7, SW41 U, SW42 J, SW43 M, SW44 F6, SW45 8, SW46 I, SW47 K, SW48 COMMA, SW49 RALT, SW5 CAPS, SW50 F7, SW51 9, SW52 O, SW53 L, SW54 DOT, SW55 FN, SW56 F8, SW57 0, SW58 P, SW59 SEMICOLON, SW6 LSHIFT, SW60 SLASH, SW61 MENU, SW62 MINUS, SW63 SQBOPEN, SW64 QUOTE, SW65 RSHIFT, SW66 RCTRL, SW67 F9, SW68 EQUAL, SW69 SQBCLOSE, SW7 LCTRL, SW70 ENTER, SW73 F10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

Commit message: setup different boards for cost reduction trial
Parts:
- added J10: key_board_conn, Connector_PinHeader_2.54mm:PinHeader_1x26_P2.54mm_Vertical, symbol Connector_Generic:Conn_01x26
- added J11: main_board_conn, Connector_PinHeader_2.54mm:PinHeader_1x26_P2.54mm_Vertical, symbol Connector_Generic:Conn_01x26
Connections:
- net COL_01: now also J10.1 (Pin_1); no longer MDBT50Q_1.13 (P0.28/AIN4)
- net COL_02: now also J10.2 (Pin_2); no longer MDBT50Q_1.14 (P0.30/AIN6)
- net COL_03: now also J10.3 (Pin_3); no longer MDBT50Q_1.16 (P0.27)
- net COL_04: now also J10.4 (Pin_4); no longer MDBT50Q_1.17 (P0.00/XL1)
- net COL_05: now also J10.5 (Pin_5); no longer MDBT50Q_1.18 (P0.01/XL2)
- net COL_06: now also J10.6 (Pin_6); no longer MDBT50Q_1.19 (P0.26)
- net COL_07: now also J10.7 (Pin_7); no longer MDBT50Q_1.20 (P0.04/AIN2)
- net COL_08: now also J10.8 (Pin_8); no longer MDBT50Q_1.21 (P0.05/AIN3)
- net COL_09: now also J10.9 (Pin_9); no longer MDBT50Q_1.22 (P0.06)
- net COL_10: now also J10.10 (Pin_10); no longer MDBT50Q_1.23 (P0.07)
- net COL_11: now also J10.11 (Pin_11); no longer MDBT50Q_1.24 (P0.08)
- net COL_12: now also J10.12 (Pin_12); no longer MDBT50Q_1.25 (P1.08)
- net COL_13: now also J10.13 (Pin_13); no longer MDBT50Q_1.26 (P1.09)
- net COL_14: now also J10.14 (Pin_14); no longer MDBT50Q_1.27 (P0.11)
- net COL_15: now also J10.15 (Pin_15); no longer MDBT50Q_1.29 (P0.12)
- net GND: now also J10.25 (Pin_25), J10.26 (Pin_26), J11.25 (Pin_25), J11.26 (Pin_26)
- net RE_A: now also J10.22 (Pin_22); no longer MDBT50Q_1.44 (P0.20)
- net RE_B: now also J10.23 (Pin_23); no longer MDBT50Q_1.43 (P0.21)
- net RE_Sw: now also J10.24 (Pin_24); no longer MDBT50Q_1.46 (P0.22)
- net ROW_01: now also J10.16 (Pin_16); no longer MDBT50Q_1.4 (P1.11)
- net ROW_02: now also J10.17 (Pin_17); no longer MDBT50Q_1.5 (P1.12)
- net ROW_03: now also J10.18 (Pin_18); no longer MDBT50Q_1.6 (P1.13)
- net ROW_04: now also J10.19 (Pin_19); no longer MDBT50Q_1.7 (P1.14)
- net ROW_05: now also J10.20 (Pin_20); no longer MDBT50Q_1.8 (P1.15)
- net ROW_06: now also J10.21 (Pin_21); no longer MDBT50Q_1.9 (P0.03/AIN1)
- new net MB_COL_01: J11.1 (Pin_1), MDBT50Q_1.4 (P1.11)
- new net MB_COL_02: J11.2 (Pin_2), MDBT50Q_1.5 (P1.12)
- new net MB_COL_03: J11.3 (Pin_3), MDBT50Q_1.6 (P1.13)
- new net MB_COL_04: J11.4 (Pin_4), MDBT50Q_1.7 (P1.14)
- new net MB_COL_05: J11.5 (Pin_5), MDBT50Q_1.8 (P1.15)
- new net MB_COL_06: J11.6 (Pin_6), MDBT50Q_1.9 (P0.03/AIN1)
- new net MB_COL_07: J11.7 (Pin_7), MDBT50Q_1.13 (P0.28/AIN4)
- new net MB_COL_08: J11.8 (Pin_8), MDBT50Q_1.14 (P0.30/AIN6)
- new net MB_COL_09: J11.9 (Pin_9), MDBT50Q_1.16 (P0.27)
- new net MB_COL_10: J11.10 (Pin_10), MDBT50Q_1.17 (P0.00/XL1)
- new net MB_COL_11: J11.11 (Pin_11), MDBT50Q_1.18 (P0.01/XL2)
- new net MB_COL_12: J11.12 (Pin_12), MDBT50Q_1.19 (P0.26)
- new net MB_COL_13: J11.13 (Pin_13), MDBT50Q_1.20 (P0.04/AIN2)
- new net MB_COL_14: J11.14 (Pin_14), MDBT50Q_1.21 (P0.05/AIN3)
- new net MB_COL_15: J11.15 (Pin_15), MDBT50Q_1.22 (P0.06)
- new net MB_RE_A: J11.22 (Pin_22), MDBT50Q_1.44 (P0.20)
- new net MB_RE_B: J11.23 (Pin_23), MDBT50Q_1.43 (P0.21)
- new net MB_RE_Sw: J11.24 (Pin_24), MDBT50Q_1.46 (P0.22)
- new net MB_ROW_01: J11.16 (Pin_16), MDBT50Q_1.23 (P0.07)
- new net MB_ROW_02: J11.17 (Pin_17), MDBT50Q_1.24 (P0.08)
- new net MB_ROW_03: J11.18 (Pin_18), MDBT50Q_1.25 (P1.08)
- new net MB_ROW_04: J11.19 (Pin_19), MDBT50Q_1.26 (P1.09)
- new net MB_ROW_05: J11.20 (Pin_20), MDBT50Q_1.27 (P0.11)
- new net MB_ROW_06: J11.21 (Pin_21), MDBT50Q_1.29 (P0.12)
Other:
- note added: "Total GPIO = 21 ROW01-06 COL01-15"
- note removed: "Total GPIO = 22 ROW01-06 COL01-16"
- moved on the sheet: D10, D11, D12, D13, D14, D15, D16, D17, D18, D19, D2, D20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

Commit message: added teardrops on daughter board
Parts:
- removed C1, C2: 1uF, Capacitor_SMD:C_0402_1005Metric, symbol Device:C_Small
- removed C3, C4: 10uF, Capacitor_SMD:C_0402_1005Metric, symbol Device:C_Small
- removed C5: 0.1uF, Capacitor_SMD:C_0402_1005Metric, symbol Device:C_Small
- removed IC1: BQ24040DSQR, BQ24040DSQR-lion:SON40P200X200X80-11N, symbol BQ24040DSQR:BQ24040DSQR
- removed IC2: TPS63031DSKR, TPS63031DSKR-lion:SON50P250X250X80-11N-D, symbol TPS63031DSKR:TPS63031DSKR
- removed J1: Display, Connector_PinHeader_2.54mm:PinHeader_1x08_P2.54mm_Vertical, symbol Connector_Generic:Conn_01x08
- removed J11: main_board_conn, Connector_PinHeader_2.54mm:PinHeader_1x26_P2.54mm_Vertical, symbol Connector_Generic:Conn_01x26
- removed J2: USB4216-03-A, USB421603A, symbol USB4216-03-A:USB4216-03-A
- removed J3: ProgConn, Connector_PinHeader_2.54mm:PinHeader_1x04_P2.54mm_Vertical, symbol Connector_Generic:Conn_01x04
- removed J4: PG_LED, Connector_PinHeader_2.54mm:PinHeader_1x02_P2.54mm_Vertical, symbol Connector_Generic:Conn_01x02
- removed J5: CHRG_LED, Connector_PinHeader_2.54mm:PinHeader_1x02_P2.54mm_Vertical, symbol Connector_Generic:Conn_01x02
- removed J6: POWER_LED, Connector_PinHeader_2.54mm:PinHeader_1x02_P2.54mm_Vertical, symbol Connector_Generic:Conn_01x02
- removed J7: Mode Selector, Connector_PinHeader_2.54mm:PinHeader_1x03_P2.54mm_Vertical, symbol Connector_Generic:Conn_01x03
- removed J8: Mode Selector, Connector_PinHeader_2.54mm:PinHeader_1x04_P2.54mm_Vertical, symbol Connector_Generic:Conn_01x04
- removed J9: LED_STRIP, Connector_PinHeader_2.54mm:PinHeader_1x03_P2.54mm_Vertical, symbol Connector_Generic:Conn_01x03
- removed L2: LPS3015-222MRC, LPS3015-222MRC:IND_LPS3015-222MRC, symbol LPS3015-222MRC:LPS3015-222MRC
- removed MDBT50Q_1: MDBT50Q_1, RF_Module:Raytac_MDBT50Q, symbol MDBT50Q-U_52840_230606:MDBT50Q_52840
- removed R1, R2: 5.1k, Resistor_SMD:R_0402_1005Metric, symbol Device:R_Small
- removed R10: 400k, Connector_PinHeader_2.54mm:PinHeader_1x02_P2.54mm_Vertical, symbol Device:R_Small
- removed R3: 1k, Connector_PinHeader_2.54mm:PinHeader_1x02_P2.54mm_Vertical, symbol Device:R_Small
- removed R4: 2k, Connector_PinHeader_2.54mm:PinHeader_1x02_P2.54mm_Vertical, symbol Device:R_Small
- removed R5: 10k, Connector_PinHeader_2.54mm:PinHeader_1x02_P2.54mm_Vertical, symbol Device:R_Small
- removed R6, R7, R8: 330, Connector_PinHeader_2.54mm:PinHeader_1x02_P2.54mm_Vertical, symbol Device:R_Small
- removed R9: 300k, Connector_PinHeader_2.54mm:PinHeader_1x02_P2.54mm_Vertical, symbol Device:R_Small
Connections:
- no-connect marks 2 -> 0
Other:
- note removed: "3.3V Voltage Regulator"
- note removed: "8x WS2812"
- note removed: "BLE / USB Mode Selector Switch"
- note removed: "Battery Charging + Power Path"
- note removed: "Display"
- note removed: "Fuel Gauge Voltage Divider"
- note removed: "LED Strip"
- note removed: "MCU"
- note removed: "Normal Voltage mode"
- note removed: "P0.13"
- note removed: "P0.14"
- note removed: "P0.15"
- note removed: "P0.16"
- note removed: "P0.17"
- note removed: "P0.19"
- note removed: "P0.31"
- note removed: "P1.00"
- note removed: "Power Path Selection"
- note removed: "Status LEDs"
- note removed: "USB-C"
- note removed: "will only be active in USB mode"
- moved on the sheet: D10, D11, D12, D13, D14, D15, D16, D17, D18, D19, D2, D20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

Commit message: pcb finish rev2
Parts:
- D10, D11, D12, D13, D14, D15, D16, D17, D18, D19, D2, D20, D21, D22, D23, D24, D25, D26, D27, D28, D29, D3, D30, D31, D32, D33, D34, D35, D36, D37, D38, D39, D4, D40, D41, D42, D43, D44, D45, D46, D47, D48, D49, D5, D50, D51, D52, D53, D54, D55, D56, D57, D58, D59, D6, D60, D61, D62, D63, D64, D65, D66, D67, D68, D69, D7, D70, D73, D74, D75, D77, D8, D81, D9: value 1N4148WS -> 1N4148TA; footprint Diode_SMD:D_SOD-323F -> Diode_THT:D_DO-35_SOD27_P7.62mm_Horizontal
