File: PCB/main_board/main_board.kicad_pcb (KiCad board)
At the start: 4 copper layers, 291.2 x 130.9 mm, 180 parts, among them IC1 BQ24040DSQR, IC2 TPS63031DSKR, J1 Display, J10 key_board_conn, J11 main_board_conn, J2 USB4216-03-A, J3 ProgConn, J4 PG_LED, J5 CHRG_LED, J6 POWER_LED, J7 Mode Selector, J8 Mode Selector, J9 LED_STRIP, SW1 RotaryEncoder_Switch, SW10 A, SW11 Z, SW12 WIN, SW13 F1, SW14 2, SW15 W, SW16 S, SW17 X, SW18 LALT, SW19 F2, SW2 ESC, SW20 3, SW21 E, SW22 D, SW23 C, SW24 SPACE, SW25 F3, SW26 4, SW27 R, SW28 F, SW29 V, SW3 TILDE, SW30 F4, SW31 5, SW32 T, SW33 G, SW34 B, SW35 6, SW36 Y, SW37 H, SW38 N, SW39 F5, SW4 TAB, SW40 7, SW41 U, SW42 J, SW43 M, SW44 F6, SW45 8, SW46 I, SW47 K, SW48 COMMA, SW49 RALT, SW5 CAPS, SW50 F7, SW51 9, SW52 O, SW53 L, SW54 DOT, SW55 FN, SW56 F8, SW57 0, SW58 P, SW59 SEMICOLON, SW6 LSHIFT, SW60 SLASH, SW61 MENU, SW62 MINUS, SW63 SQBOPEN, SW64 QUOTE, SW65 RSHIFT, SW66 RCTRL, SW67 F9, SW68 EQUAL, SW69 SQBCLOSE, SW7 LCTRL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

Commit message: main board rev1
Parts:
- removed D10, D11, D12, D13, D14, D15, D16, D17, D18, D19, D2, D20, D21, D22, D23, D24, D25, D26, D27, D28, D29, D3, D30, D31, D32, D33, D34, D35, D36, D37, D38, D39, D4, D40, D41, D42, D43, D44, D45, D46, D47, D48, D49, D5, D50, D51, D52, D53, D54, D55, D56, D57, D58, D59, D6, D60, D61, D62, D63, D64, D65, D66, D67, D68, D69, D7, D70, D73, D74, D75, D77, D8, D81, D9: 1N4148WS, Diode_SMD:D_SOD-323F
- removed G***: LOGO, LOGO
- removed SW1: RotaryEncoder_Switch, Rotary_Encoder:RotaryEncoder_Alps_EC11E-Switch_Vertical_H20mm
- removed SW10: A, Button_Switch_Keyboard:3Dfyd_SW_Cherry_MX_1.00u_PCB
- removed SW11: Z, Button_Switch_Keyboard:3Dfyd_SW_Cherry_MX_1.00u_PCB
- removed SW12: WIN, Button_Switch_Keyboard:3dfyd_SW_Cherry_MX_1.25u_PCB
- removed SW13: F1, Button_Switch_Keyboard:3Dfyd_SW_Cherry_MX_1.00u_PCB
- removed SW14: 2, Button_Switch_Keyboard:3Dfyd_SW_Cherry_MX_1.00u_PCB
- removed SW15: W, Button_Switch_Keyboard:3Dfyd_SW_Cherry_MX_1.00u_PCB
- removed SW16: S, Button_Switch_Keyboard:3Dfyd_SW_Cherry_MX_1.00u_PCB
- removed SW17: X, Button_Switch_Keyboard:3Dfyd_SW_Cherry_MX_1.00u_PCB
- removed SW18: LALT, Button_Switch_Keyboard:3dfyd_SW_Cherry_MX_1.25u_PCB
- removed SW19: F2, Button_Switch_Keyboard:3Dfyd_SW_Cherry_MX_1.00u_PCB
- removed SW2: ESC, Button_Switch_Keyboard:3Dfyd_SW_Cherry_MX_1.00u_PCB
- removed SW20: 3, Button_Switch_Keyboard:3Dfyd_SW_Cherry_MX_1.00u_PCB
- removed SW21: E, Button_Switch_Keyboard:3Dfyd_SW_Cherry_MX_1.00u_PCB
- removed SW22: D, Button_Switch_Keyboard:3Dfyd_SW_Cherry_MX_1.00u_PCB
- removed SW23: C, Button_Switch_Keyboard:3Dfyd_SW_Cherry_MX_1.00u_PCB
- removed SW24: SPACE, Button_Switch_Keyboard:3Dfyd_SW_Cherry_MX_6.25u_PCB
- removed SW25: F3, Button_Switch_Keyboard:3Dfyd_SW_Cherry_MX_1.00u_PCB
- removed SW26: 4, Button_Switch_Keyboard:3Dfyd_SW_Cherry_MX_1.00u_PCB
- removed SW27: R, Button_Switch_Keyboard:3Dfyd_SW_Cherry_MX_1.00u_PCB
- removed SW28: F, Button_Switch_Keyboard:3Dfyd_SW_Cherry_MX_1.00u_PCB
- removed SW29: V, Button_Switch_Keyboard:3Dfyd_SW_Cherry_MX_1.00u_PCB
- removed SW3: TILDE, Button_Switch_Keyboard:3Dfyd_SW_Cherry_MX_1.00u_PCB
- removed SW30: F4, Button_Switch_Keyboard:3Dfyd_SW_Cherry_MX_1.00u_PCB
- removed SW31: 5, Button_Switch_Keyboard:3Dfyd_SW_Cherry_MX_1.00u_PCB
- removed SW32: T, Button_Switch_Keyboard:3Dfyd_SW_Cherry_MX_1.00u_PCB
- removed SW33: G, Button_Switch_Keyboard:3Dfyd_SW_Cherry_MX_1.00u_PCB
- removed SW34: B, Button_Switch_Keyboard:3Dfyd_SW_Cherry_MX_1.00u_PCB
- removed SW35: 6, Button_Switch_Keyboard:3Dfyd_SW_Cherry_MX_1.00u_PCB
- removed SW36: Y, Button_Switch_Keyboard:3Dfyd_SW_Cherry_MX_1.00u_PCB
- removed SW37: H, Button_Switch_Keyboard:3Dfyd_SW_Cherry_MX_1.00u_PCB
- removed SW38: N, Button_Switch_Keyboard:3Dfyd_SW_Cherry_MX_1.00u_PCB
- removed SW39: F5, Button_Switch_Keyboard:3Dfyd_SW_Cherry_MX_1.00u_PCB
- removed SW4: TAB, Button_Switch_Keyboard:3Dfyd_SW_Cherry_MX_1.50u_PCB
- removed SW40: 7, Button_Switch_Keyboard:3Dfyd_SW_Cherry_MX_1.00u_PCB
- removed SW41: U, Button_Switch_Keyboard:3Dfyd_SW_Cherry_MX_1.00u_PCB
- removed SW42: J, Button_Switch_Keyboard:3Dfyd_SW_Cherry_MX_1.00u_PCB
- removed SW43: M, Button_Switch_Keyboard:3Dfyd_SW_Cherry_MX_1.00u_PCB
- removed SW44: F6, Button_Switch_Keyboard:3Dfyd_SW_Cherry_MX_1.00u_PCB
- removed SW45: 8, Button_Switch_Keyboard:3Dfyd_SW_Cherry_MX_1.00u_PCB
- removed SW46: I, Button_Switch_Keyboard:3Dfyd_SW_Cherry_MX_1.00u_PCB
- removed SW47: K, Button_Switch_Keyboard:3Dfyd_SW_Cherry_MX_1.00u_PCB
- removed SW48: COMMA, Button_Switch_Keyboard:3Dfyd_SW_Cherry_MX_1.00u_PCB
- removed SW49: RALT, Button_Switch_Keyboard:3dfyd_SW_Cherry_MX_1.25u_PCB
- removed SW5: CAPS, Button_Switch_Keyboard:3Dfyd_SW_Cherry_MX_1.75u_PCB
- removed SW50: F7, Button_Switch_Keyboard:3Dfyd_SW_Cherry_MX_1.00u_PCB
- removed SW51: 9, Button_Switch_Keyboard:3Dfyd_SW_Cherry_MX_1.00u_PCB
- removed SW52: O, Button_Switch_Keyboard:3Dfyd_SW_Cherry_MX_1.00u_PCB
- removed SW53: L, Button_Switch_Keyboard:3Dfyd_SW_Cherry_MX_1.00u_PCB
- removed SW54: DOT, Button_Switch_Keyboard:3Dfyd_SW_Cherry_MX_1.00u_PCB
- removed SW55: FN, Button_Switch_Keyboard:3dfyd_SW_Cherry_MX_1.25u_PCB
- removed SW56: F8, Button_Switch_Keyboard:3Dfyd_SW_Cherry_MX_1.00u_PCB
- removed SW57: 0, Button_Switch_Keyboard:3Dfyd_SW_Cherry_MX_1.00u_PCB
- removed SW58: P, Button_Switch_Keyboard:3Dfyd_SW_Cherry_MX_1.00u_PCB
- removed SW59: SEMICOLON, Button_Switch_Keyboard:3Dfyd_SW_Cherry_MX_1.00u_PCB
- removed SW6: LSHIFT, Button_Switch_Keyboard:3Dfyd_SW_Cherry_MX_2.25u_PCB
- removed SW60: SLASH, Button_Switch_Keyboard:3Dfyd_SW_Cherry_MX_1.00u_PCB
- removed SW61: MENU, Button_Switch_Keyboard:3dfyd_SW_Cherry_MX_1.25u_PCB
- removed SW62: MINUS, Button_Switch_Keyboard:3Dfyd_SW_Cherry_MX_1.00u_PCB
- removed SW63: SQBOPEN, Button_Switch_Keyboard:3Dfyd_SW_Cherry_MX_1.00u_PCB
- removed SW64: QUOTE, Button_Switch_Keyboard:3Dfyd_SW_Cherry_MX_1.00u_PCB
- removed SW65: RSHIFT, Button_Switch_Keyboard:3Dfyd_SW_Cherry_MX_2.75u_PCB
- removed SW66: RCTRL, Button_Switch_Keyboard:3dfyd_SW_Cherry_MX_1.25u_PCB
- removed SW67: F9, Button_Switch_Keyboard:3Dfyd_SW_Cherry_MX_1.00u_PCB
- removed SW68: EQUAL, Button_Switch_Keyboard:3Dfyd_SW_Cherry_MX_1.00u_PCB
- removed SW69: SQBCLOSE, Button_Switch_Keyboard:3Dfyd_SW_Cherry_MX_1.00u_PCB
- removed SW7: LCTRL, Button_Switch_Keyboard:3dfyd_SW_Cherry_MX_1.25u_PCB
- removed SW70: ENTER, Button_Switch_Keyboard:3Dfyd_SW_Cherry_MX_2.25u_PCB
- removed SW73: F10, Button_Switch_Keyboard:3Dfyd_SW_Cherry_MX_1.00u_PCB
- removed SW74: BACKSPACE, Button_Switch_Keyboard:3Dfyd_SW_Cherry_MX_2.00u_PCB
- removed SW75: FWDSLASH, Button_Switch_Keyboard:3Dfyd_SW_Cherry_MX_1.50u_PCB
- removed SW77: F11, Button_Switch_Keyboard:3Dfyd_SW_Cherry_MX_1.00u_PCB
- removed SW8: 1, Button_Switch_Keyboard:3Dfyd_SW_Cherry_MX_1.00u_PCB
- removed SW81: F12, Button_Switch_Keyboard:3Dfyd_SW_Cherry_MX_1.00u_PCB
- removed SW9: Q, Button_Switch_Keyboard:3Dfyd_SW_Cherry_MX_1.00u_PCB
- added mhole_1: MountingHole, MountingHole:MountingHole_3mm, F.Cu at (255.6, 188.3)
- added mhole_2: MountingHole, MountingHole:MountingHole_3mm, F.Cu at (334.3, 193.5)
- J10: value key_board_conn -> Conn_01x02; footprint Connector_PinHeader_2.54mm:PinHeader_1x26_P2.54mm_Vertical -> Connector_PinHeader_2.54mm:PinHeader_1x02_P2.54mm_Vertical
- moved J9 215.8 mm to (337.4, 212.0), turned to 180 degrees
- moved J8 199.4 mm to (266.7, 212.0), turned to -90 degrees
- moved R9 176.8 mm to (272.2, 198.6)
- moved R10 176.5 mm to (275.8, 198.6), turned to 90 degrees
- moved C1 169.4 mm to (277.9, 203.1), turned to -90 degrees
- moved C2 168.9 mm to (274.9, 203.6), turned to 0 degrees
- moved IC1 165.5 mm to (275.7, 201.7), turned to 180 degrees
- moved J2 165.3 mm to (253.9, 199.0), turned to -90 degrees
- moved R2 163.3 mm to (259.9, 201.0), turned to 0 degrees
- moved C3 161.7 mm to (268.1, 200.3), turned to 0 degrees
- moved C5 161.1 mm to (265.0, 204.8), turned to -90 degrees
- moved C4 160.9 mm to (268.1, 199.2), turned to 0 degrees
- moved IC2 159.3 mm to (265.5, 201.5), turned to -90 degrees
- moved R3 158.9 mm to (279.5, 192.5)
- moved R1 158.9 mm to (259.9, 197.5), turned to 0 degrees
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Connections:
- J10 pad 1: /COL_01 -> GND
- J10 pad 2: /COL_02 -> /MCU_RESET
Routing:
- net /ROW_06: track 442.4 -> 0.00 mm, vias 1 -> 0
- net /ROW_05: track 385.3 -> 0.00 mm, vias 1 -> 0
- net /ROW_04: track 365.5 -> 0.00 mm, vias 1 -> 0
- net /ROW_02: track 360.0 -> 0.00 mm, vias 1 -> 0
- net /ROW_03: track 350.6 -> 0.00 mm, vias 1 -> 0
- net /ROW_01: track 296.2 -> 0.00 mm, vias 1 -> 0
- net /COL_01: track 285.9 -> 0.00 mm
- net /COL_02: track 274.0 -> 0.00 mm, vias 1 -> 0
- net /COL_04: track 266.7 -> 0.00 mm
- net /COL_03: track 258.8 -> 0.00 mm
- net /COL_05: track 201.8 -> 0.00 mm
- net /COL_06: track 185.3 -> 0.00 mm
- net /COL_09: track 175.2 -> 0.00 mm
- net /COL_07: track 168.8 -> 0.00 mm, vias 1 -> 0
- net /COL_08: track 165.7 -> 0.00 mm
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- added copper zone on In2.Cu, net +3.3V
- added copper zone on In1.Cu, net GND
Other:
- board size 291.2 x 130.9 mm -> 88.8 x 30.7 mm
- board text added: "RESET/GND"
- board text removed: "(NOT ON PCB, WILL BE RAISED UP)"
- board text removed: "K-0"

Commit message: pcb finish rev2
Routing:
- net GND: vias 78 -> 80
Changed lines of the file:
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@@
 	)
 	(gr_text "D"
-		(at 335.7596 208.8652 90)
-		(layer "B.SilkS")
+		(at 335.84 208.85 90)
+		(layer "B.SilkS" knockout)
 		(effects
 			(font
@@
 	)
 	(gr_text "+\n"
-		(at 335.7126 206.1822 90)
-		(layer "B.SilkS")
+		(at 336.23 206.22 90)
+		(layer "B.SilkS" knockout)
 		(effects
 			(font
@@
 	)
 	(gr_text "-"
-		(at 335.7486 212.0322 90)
-		(layer "B.SilkS")
+		(at 336.26 212.0322 90)
+		(layer "B.SilkS" knockout)
 		(effects
 			(font
@@
 	)
 	(via
-		(at 289.179 200.505)
+		(at 289.16 200.37)
 		(size 0.6)
 		(drill 0.3)
@@
 	)
 	(via
-		(at 291.719 200.505)
+		(at 291.7 200.37)
 		(size 0.6)
 		(drill 0.3)
@@
 	)
 	(via
-		(at 290.449 199.235)
+		(at 290.43 199.1)
 		(size 0.6)
 		(drill 0.3)
@@
 	)
 	(via
+		(at 290.42 201.46)
+		(size 0.6)
+		(drill 0.3)
+		(layers "F.Cu" "B.Cu")
+		(net 2)
+	)
+	(via
 		(at 283.629 189.035)
 		(size 0.6)
@@
 	)
 	(via
-		(at 305.4271 205.538)
+		(at 305.85 202.8)
+		(size 0.6)
+		(drill 0.3)
+		(layers "F.Cu" "B.Cu")
+		(free yes)
+		(net 2)
+	)
+	(via
+		(at 305.08 205.539)
 		(size 0.6)
 		(drill 0.3)
@@
 	)
 	(via
-		(at 292.979 195.005)
+		(at 292.91 195.37)
 		(size 0.6)
 		(drill 0.3)
@@
 	)
 	(via
-		(at 302.4331 202.73)
+		(at 302.33 202.76)
 		(size 0.6)
 		(drill 0.3)
@@
 	)
 	(via
-		(at 290.439 195.005)
-		(size 0.6)
-		(drill 0.3)
+		(at 290.439 195.36)
+		(size 0.6)
+		(drill 0.3)
