File: PCB/main_board/main_board.kicad_sch (KiCad schematic)
At the start: 179 parts, among them IC1 BQ24040DSQR, IC2 TPS63031DSKR, J1 Display, J10 key_board_conn, J11 main_board_conn, J2 USB4216-03-A, J3 ProgConn, J4 PG_LED, J5 CHRG_LED, J6 POWER_LED, J7 Mode Selector, J8 Mode Selector, J9 LED_STRIP, SW1 RotaryEncoder_Switch, SW10 A, SW11 Z, SW12 WIN, SW13 F1, SW14 2, SW15 W, SW16 S, SW17 X, SW18 LALT, SW19 F2, SW2 ESC, SW20 3, SW21 E, SW22 D, SW23 C, SW24 SPACE, SW25 F3, SW26 4, SW27 R, SW28 F, SW29 V, SW3 TILDE, SW30 F4, SW31 5, SW32 T, SW33 G, SW34 B, SW35 6, SW36 Y, SW37 H, SW38 N, SW39 F5, SW4 TAB, SW40 7, SW41 U, SW42 J, SW43 M, SW44 F6, SW45 8, SW46 I, SW47 K, SW48 COMMA, SW49 RALT, SW5 CAPS, SW50 F7, SW51 9, SW52 O, SW53 L, SW54 DOT, SW55 FN, SW56 F8, SW57 0, SW58 P, SW59 SEMICOLON, SW6 LSHIFT, SW60 SLASH, SW61 MENU, SW62 MINUS, SW63 SQBOPEN, SW64 QUOTE, SW65 RSHIFT, SW66 RCTRL, SW67 F9, SW68 EQUAL, SW69 SQBCLOSE, SW7 LCTRL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

Commit message: main board rev1
Parts:
- removed D10, D11, D12, D13, D14, D15, D16, D17, D18, D19, D2, D20, D21, D22, D23, D24, D25, D26, D27, D28, D29, D3, D30, D31, D32, D33, D34, D35, D36, D37, D38, D39, D4, D40, D41, D42, D43, D44, D45, D46, D47, D48, D49, D5, D50, D51, D52, D53, D54, D55, D56, D57, D58, D59, D6, D60, D61, D62, D63, D64, D65, D66, D67, D68, D69, D7, D70, D73, D74, D75, D77, D8, D81, D9: 1N4148WS, Diode_SMD:D_SOD-323F, symbol Device:D_Small
- removed J10: key_board_conn, Connector_PinHeader_2.54mm:PinHeader_1x26_P2.54mm_Vertical, symbol Connector_Generic:Conn_01x26
- removed SW1: RotaryEncoder_Switch, Rotary_Encoder:RotaryEncoder_Alps_EC11E-Switch_Vertical_H20mm, symbol Device:RotaryEncoder_Switch
- removed SW10: A, Button_Switch_Keyboard:3Dfyd_SW_Cherry_MX_1.00u_PCB, symbol Switch:SW_Push
- removed SW11: Z, Button_Switch_Keyboard:3Dfyd_SW_Cherry_MX_1.00u_PCB, symbol Switch:SW_Push
- removed SW12: WIN, Button_Switch_Keyboard:3dfyd_SW_Cherry_MX_1.25u_PCB, symbol Switch:SW_Push
- removed SW13: F1, Button_Switch_Keyboard:3Dfyd_SW_Cherry_MX_1.00u_PCB, symbol Switch:SW_Push
- removed SW14: 2, Button_Switch_Keyboard:3Dfyd_SW_Cherry_MX_1.00u_PCB, symbol Switch:SW_Push
- removed SW15: W, Button_Switch_Keyboard:3Dfyd_SW_Cherry_MX_1.00u_PCB, symbol Switch:SW_Push
- removed SW16: S, Button_Switch_Keyboard:3Dfyd_SW_Cherry_MX_1.00u_PCB, symbol Switch:SW_Push
- removed SW17: X, Button_Switch_Keyboard:3Dfyd_SW_Cherry_MX_1.00u_PCB, symbol Switch:SW_Push
- removed SW18: LALT, Button_Switch_Keyboard:3dfyd_SW_Cherry_MX_1.25u_PCB, symbol Switch:SW_Push
- removed SW19: F2, Button_Switch_Keyboard:3Dfyd_SW_Cherry_MX_1.00u_PCB, symbol Switch:SW_Push
- removed SW2: ESC, Button_Switch_Keyboard:3Dfyd_SW_Cherry_MX_1.00u_PCB, symbol Switch:SW_Push
- removed SW20: 3, Button_Switch_Keyboard:3Dfyd_SW_Cherry_MX_1.00u_PCB, symbol Switch:SW_Push
- removed SW21: E, Button_Switch_Keyboard:3Dfyd_SW_Cherry_MX_1.00u_PCB, symbol Switch:SW_Push
- removed SW22: D, Button_Switch_Keyboard:3Dfyd_SW_Cherry_MX_1.00u_PCB, symbol Switch:SW_Push
- removed SW23: C, Button_Switch_Keyboard:3Dfyd_SW_Cherry_MX_1.00u_PCB, symbol Switch:SW_Push
- removed SW24: SPACE, Button_Switch_Keyboard:3Dfyd_SW_Cherry_MX_6.25u_PCB, symbol Switch:SW_Push
- removed SW25: F3, Button_Switch_Keyboard:3Dfyd_SW_Cherry_MX_1.00u_PCB, symbol Switch:SW_Push
- removed SW26: 4, Button_Switch_Keyboard:3Dfyd_SW_Cherry_MX_1.00u_PCB, symbol Switch:SW_Push
- removed SW27: R, Button_Switch_Keyboard:3Dfyd_SW_Cherry_MX_1.00u_PCB, symbol Switch:SW_Push
- removed SW28: F, Button_Switch_Keyboard:3Dfyd_SW_Cherry_MX_1.00u_PCB, symbol Switch:SW_Push
- removed SW29: V, Button_Switch_Keyboard:3Dfyd_SW_Cherry_MX_1.00u_PCB, symbol Switch:SW_Push
- removed SW3: TILDE, Button_Switch_Keyboard:3Dfyd_SW_Cherry_MX_1.00u_PCB, symbol Switch:SW_Push
- removed SW30: F4, Button_Switch_Keyboard:3Dfyd_SW_Cherry_MX_1.00u_PCB, symbol Switch:SW_Push
- removed SW31: 5, Button_Switch_Keyboard:3Dfyd_SW_Cherry_MX_1.00u_PCB, symbol Switch:SW_Push
- removed SW32: T, Button_Switch_Keyboard:3Dfyd_SW_Cherry_MX_1.00u_PCB, symbol Switch:SW_Push
- removed SW33: G, Button_Switch_Keyboard:3Dfyd_SW_Cherry_MX_1.00u_PCB, symbol Switch:SW_Push
- removed SW34: B, Button_Switch_Keyboard:3Dfyd_SW_Cherry_MX_1.00u_PCB, symbol Switch:SW_Push
- removed SW35: 6, Button_Switch_Keyboard:3Dfyd_SW_Cherry_MX_1.00u_PCB, symbol Switch:SW_Push
- removed SW36: Y, Button_Switch_Keyboard:3Dfyd_SW_Cherry_MX_1.00u_PCB, symbol Switch:SW_Push
- removed SW37: H, Button_Switch_Keyboard:3Dfyd_SW_Cherry_MX_1.00u_PCB, symbol Switch:SW_Push
- removed SW38: N, Button_Switch_Keyboard:3Dfyd_SW_Cherry_MX_1.00u_PCB, symbol Switch:SW_Push
- removed SW39: F5, Button_Switch_Keyboard:3Dfyd_SW_Cherry_MX_1.00u_PCB, symbol Switch:SW_Push
- removed SW4: TAB, Button_Switch_Keyboard:3Dfyd_SW_Cherry_MX_1.50u_PCB, symbol Switch:SW_Push
- removed SW40: 7, Button_Switch_Keyboard:3Dfyd_SW_Cherry_MX_1.00u_PCB, symbol Switch:SW_Push
- removed SW41: U, Button_Switch_Keyboard:3Dfyd_SW_Cherry_MX_1.00u_PCB, symbol Switch:SW_Push
- removed SW42: J, Button_Switch_Keyboard:3Dfyd_SW_Cherry_MX_1.00u_PCB, symbol Switch:SW_Push
- removed SW43: M, Button_Switch_Keyboard:3Dfyd_SW_Cherry_MX_1.00u_PCB, symbol Switch:SW_Push
- removed SW44: F6, Button_Switch_Keyboard:3Dfyd_SW_Cherry_MX_1.00u_PCB, symbol Switch:SW_Push
- removed SW45: 8, Button_Switch_Keyboard:3Dfyd_SW_Cherry_MX_1.00u_PCB, symbol Switch:SW_Push
- removed SW46: I, Button_Switch_Keyboard:3Dfyd_SW_Cherry_MX_1.00u_PCB, symbol Switch:SW_Push
- removed SW47: K, Button_Switch_Keyboard:3Dfyd_SW_Cherry_MX_1.00u_PCB, symbol Switch:SW_Push
- removed SW48: COMMA, Button_Switch_Keyboard:3Dfyd_SW_Cherry_MX_1.00u_PCB, symbol Switch:SW_Push
- removed SW49: RALT, Button_Switch_Keyboard:3dfyd_SW_Cherry_MX_1.25u_PCB, symbol Switch:SW_Push
- removed SW5: CAPS, Button_Switch_Keyboard:3Dfyd_SW_Cherry_MX_1.75u_PCB, symbol Switch:SW_Push
- removed SW50: F7, Button_Switch_Keyboard:3Dfyd_SW_Cherry_MX_1.00u_PCB, symbol Switch:SW_Push
- removed SW51: 9, Button_Switch_Keyboard:3Dfyd_SW_Cherry_MX_1.00u_PCB, symbol Switch:SW_Push
- removed SW52: O, Button_Switch_Keyboard:3Dfyd_SW_Cherry_MX_1.00u_PCB, symbol Switch:SW_Push
- removed SW53: L, Button_Switch_Keyboard:3Dfyd_SW_Cherry_MX_1.00u_PCB, symbol Switch:SW_Push
- removed SW54: DOT, Button_Switch_Keyboard:3Dfyd_SW_Cherry_MX_1.00u_PCB, symbol Switch:SW_Push
- removed SW55: FN, Button_Switch_Keyboard:3dfyd_SW_Cherry_MX_1.25u_PCB, symbol Switch:SW_Push
- removed SW56: F8, Button_Switch_Keyboard:3Dfyd_SW_Cherry_MX_1.00u_PCB, symbol Switch:SW_Push
- removed SW57: 0, Button_Switch_Keyboard:3Dfyd_SW_Cherry_MX_1.00u_PCB, symbol Switch:SW_Push
- removed SW58: P, Button_Switch_Keyboard:3Dfyd_SW_Cherry_MX_1.00u_PCB, symbol Switch:SW_Push
- removed SW59: SEMICOLON, Button_Switch_Keyboard:3Dfyd_SW_Cherry_MX_1.00u_PCB, symbol Switch:SW_Push
- removed SW6: LSHIFT, Button_Switch_Keyboard:3Dfyd_SW_Cherry_MX_2.25u_PCB, symbol Switch:SW_Push
- removed SW60: SLASH, Button_Switch_Keyboard:3Dfyd_SW_Cherry_MX_1.00u_PCB, symbol Switch:SW_Push
- removed SW61: MENU, Button_Switch_Keyboard:3dfyd_SW_Cherry_MX_1.25u_PCB, symbol Switch:SW_Push
- removed SW62: MINUS, Button_Switch_Keyboard:3Dfyd_SW_Cherry_MX_1.00u_PCB, symbol Switch:SW_Push
- removed SW63: SQBOPEN, Button_Switch_Keyboard:3Dfyd_SW_Cherry_MX_1.00u_PCB, symbol Switch:SW_Push
- removed SW64: QUOTE, Button_Switch_Keyboard:3Dfyd_SW_Cherry_MX_1.00u_PCB, symbol Switch:SW_Push
- removed SW65: RSHIFT, Button_Switch_Keyboard:3Dfyd_SW_Cherry_MX_2.75u_PCB, symbol Switch:SW_Push
- removed SW66: RCTRL, Button_Switch_Keyboard:3dfyd_SW_Cherry_MX_1.25u_PCB, symbol Switch:SW_Push
- removed SW67: F9, Button_Switch_Keyboard:3Dfyd_SW_Cherry_MX_1.00u_PCB, symbol Switch:SW_Push
- removed SW68: EQUAL, Button_Switch_Keyboard:3Dfyd_SW_Cherry_MX_1.00u_PCB, symbol Switch:SW_Push
- removed SW69: SQBCLOSE, Button_Switch_Keyboard:3Dfyd_SW_Cherry_MX_1.00u_PCB, symbol Switch:SW_Push
- removed SW7: LCTRL, Button_Switch_Keyboard:3dfyd_SW_Cherry_MX_1.25u_PCB, symbol Switch:SW_Push
- removed SW70: ENTER, Button_Switch_Keyboard:3Dfyd_SW_Cherry_MX_2.25u_PCB, symbol Switch:SW_Push
- removed SW73: F10, Button_Switch_Keyboard:3Dfyd_SW_Cherry_MX_1.00u_PCB, symbol Switch:SW_Push
- removed SW74: BACKSPACE, Button_Switch_Keyboard:3Dfyd_SW_Cherry_MX_2.00u_PCB, symbol Switch:SW_Push
- removed SW75: FWDSLASH, Button_Switch_Keyboard:3Dfyd_SW_Cherry_MX_1.50u_PCB, symbol Switch:SW_Push
- removed SW77: F11, Button_Switch_Keyboard:3Dfyd_SW_Cherry_MX_1.00u_PCB, symbol Switch:SW_Push
- removed SW8: 1, Button_Switch_Keyboard:3Dfyd_SW_Cherry_MX_1.00u_PCB, symbol Switch:SW_Push
- removed SW81: F12, Button_Switch_Keyboard:3Dfyd_SW_Cherry_MX_1.00u_PCB, symbol Switch:SW_Push
- removed SW9: Q, Button_Switch_Keyboard:3Dfyd_SW_Cherry_MX_1.00u_PCB, symbol Switch:SW_Push
- added J10: Conn_01x02, Connector_PinHeader_2.54mm:PinHeader_1x02_P2.54mm_Vertical, symbol Connector_Generic:Conn_01x02
- added mhole_1, mhole_2: MountingHole, MountingHole:MountingHole_3mm, symbol Mechanical:MountingHole
Connections:
- net GND: now also J10.1 (Pin_1)
- net MCU_RESET: now also J10.2 (Pin_2)
Other:
- note removed: "Keys Matrix"
- note removed: "P0.20"
- note removed: "P0.21"
- note removed: "P0.22"
- note removed: "Total GPIO = 21 ROW01-06 COL01-15"
- note removed: "Volume Knob"
- moved on the sheet: C1, C2, C3, C4, C5, IC1, IC2, J11, J2, J3, J4, J5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
